File: stm32devmini/stm32devmini.kicad_pcb (KiCad board)
At the start: 2 copper layers, 52.1 x 20.3 mm, 30 parts, among them J1 USB_B_Micro, SW1 SW_Push, U1 AMS1117-3.3, U2 STM32F103C8Tx, Y1 8M, Y2 32.768k

Commit message: Hmmmm
Parts:
- moved Y2 7.62 mm to (167.6, 98.4), turned to 180 degrees
- moved C11 6.98 mm to (170.8, 99.1), turned to 270 degrees
- moved C10 5.08 mm to (164.5, 101.6), turned to 270 degrees
- moved C8 2.54 mm to (164.5, 104.1)
- moved C9 2.54 mm to (164.5, 106.7)
- moved Y1 2.54 mm to (167.6, 103.5)
Routing:
- net +3V3: track 16.5 -> 50.7 mm
- net C13: track 0.00 -> 25.4 mm, vias 0 -> 2
- net A11: track 6.83 -> 25.4 mm, vias 1 -> 2
- net A12: track 6.37 -> 24.1 mm, vias 1 -> 2
- net Net-(C8-Pad1): track 0.00 -> 12.3 mm
- net Net-(C9-Pad1): track 0.00 -> 11.0 mm
- net C14: track 17.3 -> 8.44 mm
- net C15: track 15.0 -> 11.0 mm
Other:
- outline, holes or cut-outs redrawn
