File: stm32devmini/stm32devmini.kicad_pcb (KiCad board)
At the start: 2 copper layers, 52.1 x 20.3 mm, 30 parts, among them J1 USB_B_Micro, SW1 SW_Push, U1 AMS1117-3.3, U2 STM32F103C8Tx, Y1 8M, Y2 32.768k

Commit message: Hmmmm
Parts:
- J1: value USB_B_Micro -> USB_C_Receptacle_USB2.0; footprint Connector_USB:USB_Micro-B_Molex-105017-0001 -> Connector_USB:USB_C_Receptacle_HRO_TYPE-C-31-M-12
- moved R4 20.2 mm to (184.8, 106.0), turned to 270 degrees
- moved R2 17.6 mm to (209.1, 114.9)
- moved R6 17.6 mm to (210.2, 111.1)
- moved D2 16.8 mm to (184.8, 103.5), turned to 90 degrees
- moved R1 16.2 mm to (203.8, 115.6)
- moved R5 13.7 mm to (183.5, 101.6), turned to 270 degrees
- moved D3 12.7 mm to (184.8, 100.3), turned to 270 degrees
- moved D1 8.98 mm to (194.3, 101.0), turned to 90 degrees
- moved C11 6.84 mm to (164.5, 101.6)
- moved C10 6.35 mm to (168.3, 96.5), turned to 180 degrees
- moved C2 3.86 mm to (182.9, 104.8)
- moved C6 3.56 mm to (170.2, 98.4)
- moved C5 3.02 mm to (170.3, 106.0)
- moved U1 2.54 mm to (189.2, 102.9)
- moved C1 2.54 mm to (194.3, 105.4)
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Connections:
- J2 pad 1: Net-(J2-Pad1) -> VBUS
- J2 pad 17: Net-(J2-Pad17) -> RST
- J2 pad 18: Net-(J2-Pad18) -> +3V3
- J2 pad 19: Net-(J2-Pad19) -> GND
- J2 pad 20: Net-(J2-Pad20) -> GND
- R1 pad 1: Net-(J1-Pad3) -> Net-(R1-Pad1)
- R1 pad 2: A12 -> Net-(R1-Pad2)
- R2 pad 1: Net-(J1-Pad2) -> Net-(R2-Pad1)
- R2 pad 2: A11 -> Net-(R2-Pad2)
- R6 pad 2: Net-(J1-Pad3) -> Net-(R1-Pad1)
Routing:
- net A11: track 25.4 -> 37.4 mm
- net C13: track 25.4 -> 14.6 mm
- net A12: track 24.1 -> 33.7 mm
- net +3V3: track 50.7 -> 41.3 mm
- net Net-(D1-Pad2): track 14.6 -> 9.61 mm
- net Net-(J1-Pad3): track 4.43 -> 0.00 mm
- net B11: track 12.2 -> 15.6 mm
- net B10: track 9.91 -> 13.2 mm
- net B1: track 7.78 -> 10.5 mm
- net VBUS: track 5.48 -> 8.07 mm
- net Net-(J1-Pad2): track 2.50 -> 0.00 mm
- net B0: track 5.98 -> 8.09 mm
- net B12: track 22.0 -> 23.9 mm
- net A8: track 12.7 -> 14.6 mm
- net A2: track 9.02 -> 7.12 mm
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
Commit message: Hmmm
Parts:
- removed R2: 22R, Resistor_SMD:R_0402_1005Metric
- R1: value 22R -> 5.1k
- R6: value 10k -> 5.1k
- moved R1 21.7 mm to (191.8, 97.5)
- moved R6 20.9 mm to (194.3, 97.5)
Connections:
- R1 pad 1: Net-(R1-Pad1) -> Net-(J1-PadA5)
- R1 pad 2: Net-(R1-Pad2) -> GND
- R6 pad 1: Net-(D1-Pad2) -> Net-(J1-PadB5)
- R6 pad 2: Net-(R1-Pad1) -> GND
Routing:
- net VBUS: track 8.07 -> 68.8 mm
- net +3V3: track 41.3 -> 98.3 mm
- net Net-(J1-PadA5): track 0.00 -> 18.8 mm
- net C15: track 10.3 -> 23.8 mm
- net RST: track 0.00 -> 10.5 mm
- net Net-(J1-PadB5): track 0.00 -> 9.80 mm
- net Net-(D2-Pad1): track 0.00 -> 1.27 mm
- net A3: track 6.58 -> 7.09 mm
- net GND: vias 0 -> 3
Other:
- board text added: "3V3"
- board text added: "A0"
- board text added: "A1"
- board text added: "A10"
- board text added: "A11"
- board text added: "A12"
- board text added: "A15"
- board text added: "A2"
- board text added: "A3"
- board text added: "A4"
- board text added: "A5"
- board text added: "A6"
- board text added: "A7"
- board text added: "B0"
- board text added: "B1"
- board text added: "B10"
- board text added: "B11"
- board text added: "B12"
- board text added: "B13"
- board text added: "B14"
- board text added: "B15"
- board text added: "B3"
- board text added: "B4"
- board text added: "B5"
- board text added: "B6"
- board text added: "B7"
- board text added: "B8"
- board text added: "B9"
- board text added: "C13"
- board text added: "C14"
- board text added: "C15"
- board text added: "GND"
- board text added: "RST"
- board text added: "VB"

Commit message: Hmmm
Connections:
- J3 pad 1: Net-(J3-Pad1) -> +3V3
- J3 pad 2: Net-(J3-Pad2) -> GND
- J3 pad 3: Net-(J3-Pad3) -> VBUS
Routing:
- net RST: track 10.5 -> 49.1 mm, vias 0 -> 2
- net BO1: track 0.00 -> 33.1 mm, vias 0 -> 2
- net SWDIO: track 0.00 -> 32.2 mm, vias 0 -> 1
- net +3V3: track 98.3 -> 128.3 mm
- net C13: track 14.6 -> 43.6 mm
- net BO0: track 0.00 -> 28.5 mm, vias 0 -> 1
- net SWCLK: track 0.00 -> 28.4 mm, vias 0 -> 1
- net C14: track 10.1 -> 30.3 mm, vias 0 -> 1
- net VBUS: track 68.8 -> 83.9 mm
- net Net-(J1-PadA5): track 18.8 -> 17.1 mm
- net C15: track 23.8 -> 25.0 mm
- net Net-(D1-Pad2): track 9.59 -> 9.07 mm
- net GND: track 0.00 -> 0.02 mm, vias 3 -> 14
Other:
- board text added: "A8"
- board text added: "BO0"
- board text added: "BO1"
- board text added: "Black Pill Bis, rev. a STM32 Development © 2020 Lars Boegild Thomsen"
- board text added: "JLCJLCJLCJLC"

Commit message: Hmmmm
Parts:
- moved C5 1.29 mm to (171.4, 106.7)
Routing:
- net +3V3: track 128.3 -> 127.5 mm

Commit message: Hmmm
Parts:
- removed J4: ~, Connector_PinHeader_2.54mm:PinHeader_2x03_P2.54mm_Vertical
- added C12: 100nF, Capacitor_SMD:C_0402_1005Metric, F.Cu at (164.5, 102.9)
- added JP1: ~, Jumper:SolderJumper-3_P1.3mm_Open_Pad1.0x1.5mm, B.Cu at (180.9, 104.8)
- added R2: 10k, Resistor_SMD:R_0402_1005Metric, F.Cu at (164.5, 106.0)
- added SW2: ~, Button_Switch_SMD:SW_SPST_TL3342, F.Cu at (159.4, 104.8)
- SW1: value SW_Push -> ~
- U1: value AMS1117-3.3 -> XC6206P332MR; footprint Package_TO_SOT_SMD:SOT-223-3_TabPin2 -> Package_TO_SOT_SMD:SOT-23
- moved R4 7.41 mm to (188.6, 99.7), turned to 180 degrees
- moved D2 7.41 mm to (191.1, 99.7), turned to 0 degrees
- moved D3 6.63 mm to (191.1, 102.2), turned to 0 degrees
- moved R5 5.12 mm to (188.6, 102.2), turned to 180 degrees
- moved C2 5.12 mm to (188.0, 105.4)
- moved C10 4.58 mm to (172.1, 99.1), turned to 90 degrees
- moved C6 4.07 mm to (172.7, 101.6)
- moved C3 3.81 mm to (186.1, 101.6)
- moved C11 3.59 mm to (167.0, 99.1), turned to 90 degrees
- moved C4 3.33 mm to (182.2, 95.9)
- moved C5 3.24 mm to (174.6, 106.0)
- moved C8 3.17 mm to (167.0, 102.2)
- moved U1 3.17 mm to (191.1, 105.4), turned to 270 degrees
- moved U2 3.17 mm to (179.1, 101.6)
- moved C9 2.62 mm to (167.0, 106.0), turned to 90 degrees
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Routing:
- net +3V3: track 127.5 -> 0.00 mm, vias 9 -> 0
- net VBUS: track 83.9 -> 0.00 mm
- net RST: track 49.1 -> 0.00 mm, vias 2 -> 0
- net C13: track 43.4 -> 0.00 mm, vias 2 -> 0
- net BO1: track 33.1 -> 0.00 mm, vias 2 -> 0
- net SWDIO: track 31.9 -> 0.00 mm, vias 1 -> 0
- net A11: track 37.4 -> 5.87 mm
- net C14: track 30.3 -> 0.00 mm, vias 1 -> 0
- net BO0: track 28.2 -> 0.00 mm, vias 1 -> 0
- net A12: track 34.0 -> 5.90 mm
- net SWCLK: track 28.0 -> 0.00 mm, vias 1 -> 0
- net C15: track 25.0 -> 0.00 mm
- net B12: track 23.9 -> 0.00 mm
- net B13: track 21.6 -> 0.00 mm
- net B14: track 19.2 -> 0.00 mm
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- removed copper zone on B.Cu, net +3V3
- removed copper zone on F.Cu, net +3V3

Commit message: hmmmm
Routing:
- net B12: track 0.00 -> 20.7 mm
- net B13: track 0.00 -> 18.4 mm
- net Net-(J1-PadA5): track 0.00 -> 18.1 mm
- net B14: track 0.00 -> 16.0 mm
- net B15: track 0.00 -> 13.7 mm
- net A8: track 0.00 -> 11.4 mm
- net Net-(J1-PadB5): track 0.00 -> 10.3 mm
- net VBUS: track 0.00 -> 9.10 mm
- net Net-(D1-Pad2): track 0.00 -> 8.95 mm
- net A11: track 5.87 -> 11.1 mm
- net A12: track 5.90 -> 11.0 mm
- net GND: vias 0 -> 7

Commit message: Almost ready
Parts:
- removed R2, R3: 10k, Resistor_SMD:R_0402_1005Metric
- moved C7 6.98 mm to (164.5, 103.5), turned to 270 degrees
- moved SW1 6.35 mm to (159.4, 104.8), turned to 180 degrees
- moved SW2 6.35 mm to (159.4, 98.4), turned to 180 degrees
- moved JP1 4.52 mm to (185.4, 104.1), turned to 180 degrees
- moved C12 3.18 mm to (164.5, 99.7), turned to 270 degrees
- moved C10 0.64 mm to (171.4, 99.1)
- moved C11 0.63 mm to (166.4, 99.1)
- moved C8 0.63 mm to (166.4, 102.2)
- moved C9 0.63 mm to (166.4, 106.0)
- moved Y1 0.63 mm to (168.9, 104.1)
- moved Y2 0.63 mm to (168.9, 99.1)
Routing:
- net +3V3: track 0.00 -> 147.1 mm, vias 0 -> 2
- net RST: track 0.00 -> 72.0 mm, vias 0 -> 2
- net VBUS: track 9.10 -> 75.2 mm, vias 0 -> 1
- net C13: track 0.00 -> 41.9 mm, vias 0 -> 2
- net C14: track 0.00 -> 31.7 mm
- net SWDIO: track 0.00 -> 30.8 mm, vias 0 -> 1
- net SWCLK: track 0.00 -> 28.2 mm, vias 0 -> 1
- net A11: track 11.1 -> 35.2 mm
- net C15: track 0.00 -> 24.0 mm
- net A12: track 11.0 -> 34.9 mm
- net BO0: track 0.00 -> 23.7 mm, vias 0 -> 2
- net B9: track 0.00 -> 16.0 mm
- net A0: track 0.00 -> 15.0 mm
- net B8: track 0.00 -> 13.7 mm
- net A1: track 0.00 -> 12.6 mm
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Other:
- board text added: "Boot 1"
- board text added: "CLK"
- board text added: "Green Pill Bis, rev. a STM32 Development © 2020 Lars Boegild Thomsen"
- board text added: "IO"
- board text removed: "BO0"
- board text removed: "BO1"
- board text removed: "Black Pill Bis, rev. a STM32 Development © 2020 Lars Boegild Thomsen"

Commit message: Hmmm
Routing:
- net A11: track 35.2 -> 36.3 mm
- net A12: track 34.9 -> 34.0 mm
- net A10: track 7.25 -> 7.78 mm
