File: stm32devmini/stm32devmini.kicad_pcb (KiCad board)
At the start: 2 copper layers, 52.1 x 20.3 mm, 30 parts, among them J1 USB_C_Receptacle_USB2.0, U1 XC6206P332MR, U2 STM32F103C8Tx, Y1 8M, Y2 32.768k

Commit message: Hmm
Parts:
- added R1: 22R, Resistor_SMD:R_0402_1005Metric, F.Cu at (207.6, 102.2)
- added R2: 22R, Resistor_SMD:R_0402_1005Metric, F.Cu at (207.6, 104.2)
- added R3: 1.5k, Resistor_SMD:R_0402_1005Metric, F.Cu at (210.6, 102.2)
- U2: value STM32F103C8Tx -> STM32F103C8T6
- renumbered C6 to C10, C10 to C11, C11 to C12, C7 to C3, C12 to C4, C8 to C5, C3 to C6, C9 to C7, C4 to C8, C5 to C9, J5 to J4, R6 to R4, R1 to R5, R4 to R6, R5 to R7
Connections:
- C1 pad 1: VBUS -> +5V
- D1 pad 1: VBUS -> +5V
- D1 pad 2: Net-(D1-Pad2) -> VBUS
- J1 pad A4: Net-(D1-Pad2) -> VBUS
- J1 pad A6: A12 -> Net-(J1-PadA6)
- J1 pad A7: A11 -> Net-(J1-PadA7)
- J1 pad A9: Net-(D1-Pad2) -> VBUS
- J1 pad B4: Net-(D1-Pad2) -> VBUS
- J1 pad B6: A12 -> Net-(J1-PadA6)
- J1 pad B7: A11 -> Net-(J1-PadA7)
- J1 pad B9: Net-(D1-Pad2) -> VBUS
- J2 pad 1: VBUS -> +5V
- J3 pad 3: VBUS -> +5V
- U1 pad 3: VBUS -> +5V
Routing:
- net +5V: track 0.00 -> 75.2 mm, vias 0 -> 1
- net VBUS: track 75.2 -> 8.95 mm, vias 1 -> 0
- net Net-(D1-Pad2): track 8.95 -> 0.00 mm

Commit message: Hmmm
Parts:
- removed JP1: ~, Jumper:SolderJumper-3_P1.3mm_Open_Pad1.0x1.5mm
- J1: moved to B.Cu
- moved R3 9.92 mm to (200.7, 102.9)
- moved R4 9.16 mm to (200.7, 104.1), turned to 0 degrees
- moved R5 9.02 mm to (200.7, 99.1), turned to 0 degrees
- moved R2 7.46 mm to (200.7, 101.6)
- moved R1 7.24 mm to (200.7, 100.3)
- turned J1 to 270 degrees
Connections:
- J2 pad 1: +5V -> GND
- J2 pad 15: B10 -> B2
- J2 pad 16: B11 -> B10
- J2 pad 17: RST -> B11
- J2 pad 19: GND -> +5V
- J3 pad 1: +3V3 -> GND
- J3 pad 2: GND -> RST
- J3 pad 3: +5V -> BO0
- U2 pad 20: BO1 -> B2
Routing:
- net +5V: track 75.2 -> 15.4 mm, vias 1 -> 0
- net RST: track 72.0 -> 34.2 mm, vias 2 -> 3
- net Net-(J1-PadA5): track 18.8 -> 3.46 mm, vias 0 -> 1
- net B2: track 0.00 -> 8.84 mm
- net Net-(J1-PadB5): track 11.6 -> 3.25 mm, vias 0 -> 1
- net A11: track 36.3 -> 28.0 mm
- net Net-(J1-PadA6): track 0.00 -> 7.44 mm, vias 0 -> 1
- net BO0: track 23.7 -> 30.3 mm, vias 2 -> 3
- net BO1: track 6.44 -> 0.00 mm, vias 1 -> 0
- net Net-(J1-PadA7): track 0.00 -> 5.22 mm, vias 0 -> 1
- net +3V3: track 147.1 -> 151.7 mm, vias 2 -> 3
- net A12: track 34.0 -> 30.6 mm
- net VBUS: track 8.95 -> 11.9 mm, vias 0 -> 2
- net B11: track 11.0 -> 13.6 mm
- net B10: track 8.70 -> 11.2 mm
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Other:
- board text added: "5V"
- board text added: "B2"
- board text added: "BO0"
- board text removed: "VB"

Commit message: stdm rev a
Other:
- board text removed: "Boot 1"
Changed lines of the file:
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@@
   (general
     (thickness 1.2)
-    (drawings 102)
+    (drawings 103)
     (tracks 449)
     (zones 0)
@@
     )
   )
-  (gr_text 3V3 (at 154.305 105.41 90) (layer F.SilkS)
+  (gr_text 3V3 (at 154.94 105.41 90) (layer B.SilkS)
+    (effects (font (size 0.8 0.8) (thickness 0.15)) (justify mirror))
+  )
+  (gr_text IO (at 154.94 102.87 90) (layer B.SilkS)
+    (effects (font (size 0.8 0.8) (thickness 0.15)) (justify mirror))
+  )
+  (gr_text CLK (at 154.94 100.33 90) (layer B.SilkS)
+    (effects (font (size 0.8 0.8) (thickness 0.15)) (justify mirror))
+  )
+  (gr_text GND (at 154.94 97.79 90) (layer B.SilkS)
+    (effects (font (size 0.8 0.8) (thickness 0.15)) (justify mirror))
+  )
+  (gr_text 3V3 (at 154.94 105.41 90) (layer F.SilkS)
     (effects (font (size 0.8 0.8) (thickness 0.15)))
   )
-  (gr_text IO (at 154.305 102.87 90) (layer F.SilkS)
+  (gr_text IO (at 154.94 102.87 90) (layer F.SilkS)
     (effects (font (size 0.8 0.8) (thickness 0.15)))
   )
-  (gr_text CLK (at 154.305 100.33 90) (layer F.SilkS)
+  (gr_text CLK (at 154.94 100.33 90) (layer F.SilkS)
     (effects (font (size 0.8 0.8) (thickness 0.15)))
   )
-  (gr_text GND (at 154.305 97.79 90) (layer F.SilkS)
+  (gr_text GND (at 154.94 97.79 90) (layer F.SilkS)
     (effects (font (size 0.8 0.8) (thickness 0.15)))
   )
@@
     (effects (font (size 0.8 0.8) (thickness 0.15)))
   )
-  (gr_text 3V3 (at 188.595 104.14) (layer B.SilkS)
-    (effects (font (size 0.8 0.8) (thickness 0.15)) (justify mirror))
-  )
-  (gr_text GND (at 182.245 104.14) (layer B.SilkS)
-    (effects (font (size 0.8 0.8) (thickness 0.15)) (justify mirror))
-  )
-  (gr_text "Boot 1" (at 185.42 106.045) (layer B.SilkS)
-    (effects (font (size 0.8 0.8) (thickness 0.15)) (justify mirror))
-  )
   (gr_text JLCJLCJLCJLC (at 173.355 96.52) (layer B.SilkS)
