File: stm32devmini/stm32devmini.sch (KiCad schematic (older format))
At the start: 30 parts, among them J1 USB_B_Micro, SW1 SW_Push, U1 AMS1117-3.3, U2 STM32F103C8Tx, Y1 8M, Y2 32.768k

Commit message: Hmmmm
Parts:
- removed J1: USB_B_Micro, Connector_USB:USB_Micro-B_Molex-105017-0001, symbol Connector:USB_B_Micro
- added J1: USB_C_Receptacle_USB2.0, Connector_USB:USB_C_Receptacle_HRO_TYPE-C-31-M-12, symbol Connector:USB_C_Receptacle_USB2.0
Connections:
- wire segments 182 -> 190
Other:
- moved on the sheet: C1, C10, C11, C2, C3, C4, C5, C6, C8, C9, D1, J3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

Commit message: Hmmm
Parts:
- removed R2: 22R, Resistor_SMD:R_0402_1005Metric, symbol Device:R
- R1: value 22R -> 5.1k; LCSC C25092 -> C25905
- R6: value 10k -> 5.1k; LCSC C25744 -> C25905
Connections:
- wire segments 190 -> 192
Other:
- moved on the sheet: R6
Changed lines of the file:
@@
-$EndComp
-$Comp
-L Device:R R1
-U 1 1 5EF6081E
-P 3000 2050
-F 0 "R1" V 3050 2200 50  0000 C CNN
-F 1 "22R" V 3050 1850 50  0000 C CNN
-F 2 "Resistor_SMD:R_0402_1005Metric" V 2930 2050 50  0001 C CNN
-F 3 "~" H 3000 2050 50  0001 C CNN
-F 4 "C25092" V 3000 2050 50  0001 C CNN "LCSC"
-	1    3000 2050
-	0    -1   -1   0
-$EndComp
-$Comp
-L Device:R R2
-U 1 1 5EF6CBA7
-P 3000 2150
-F 0 "R2" V 3050 2300 50  0000 C CNN
-F 1 "22R" V 3050 1950 50  0000 C CNN
-F 2 "Resistor_SMD:R_0402_1005Metric" V 2930 2150 50  0001 C CNN
-F 3 "~" H 3000 2150 50  0001 C CNN
-F 4 "C25092" V 3000 2150 50  0001 C CNN "LCSC"
-	1    3000 2150
-	0    -1   -1   0
 $EndComp
 $Comp
@@
 L Device:R R6
 U 1 1 5EFA4627
-P 2600 1600
-F 0 "R6" H 2670 1646 50  0000 L CNN
-F 1 "10k" H 2670 1555 50  0000 L CNN
-F 2 "Resistor_SMD:R_0402_1005Metric" V 2530 1600 50  0001 C CNN
-F 3 "~" H 2600 1600 50  0001 C CNN
-F 4 "C25744" H 2600 1600 50  0001 C CNN "LCSC"
-	1    2600 1600
-	1    0    0    -1
-$EndComp
-Wire Wire Line
-	2600 1450 2600 1100
-Connection ~ 2600 1100
-Wire Wire Line
-	2600 1100 3000 1100
-Wire Wire Line
-	2600 1750 2600 2050
-Wire Wire Line
-	2600 2050 2850 2050
+P 2200 1650
+F 0 "R6" H 2200 1800 50  0000 L CNN
+F 1 "5.1k" H 2200 1500 50  0000 L CNN
+F 2 "Resistor_SMD:R_0402_1005Metric" V 2130 1650 50  0001 C CNN
+F 3 "~" H 2200 1650 50  0001 C CNN
+F 4 "C25905" H 2200 1650 50  0001 C CNN "LCSC"
+	1    2200 1650
+	1    0    0    -1
+$EndComp
 $Comp
 L power:+3.3V #PWR0121
@@
 $EndComp
 Wire Wire Line
-	1600 1100 2600 1100
-Wire Wire Line
 	1600 1700 1700 1700
 Wire Wire Line
@@
 Wire Wire Line
 	10450 2800 10450 2700
+$Comp
+L Device:R R1
+U 1 1 5EF5EBD1
+P 2400 1650
+F 0 "R1" H 2400 1800 50  0000 L CNN
+F 1 "5.1k" H 2400 1500 50  0000 L CNN
+F 2 "Resistor_SMD:R_0402_1005Metric" V 2330 1650 50  0001 C CNN
+F 3 "~" H 2400 1650 50  0001 C CNN
+F 4 "C25905" H 2400 1650 50  0001 C CNN "LCSC"
+	1    2400 1650
+	1    0    0    -1
+$EndComp
+$Comp
+L power:GND #PWR0131
+U 1 1 5EF5F11B
+P 2200 1900
+F 0 "#PWR0131" H 2200 1650 50  0001 C CNN
+F 1 "GND" H 2205 1727 50  0000 C CNN
+F 2 "" H 2200 1900 50  0001 C CNN
+F 3 "" H 2200 1900 50  0001 C CNN
+	1    2200 1900
+	1    0    0    -1
+$EndComp
+$Comp
+L power:GND #PWR0132
+U 1 1 5EF5F5EE
+P 2400 1900
+F 0 "#PWR0132" H 2400 1650 50  0001 C CNN
+F 1 "GND" H 2405 1727 50  0000 C CNN
+F 2 "" H 2400 1900 50  0001 C CNN
+F 3 "" H 2400 1900 50  0001 C CNN
+	1    2400 1900
+	1    0    0    -1
+$EndComp
+Wire Wire Line
+	1600 1100 3000 1100
+Wire Wire Line
+	2200 1800 2200 1900
+Wire Wire Line
+	2400 1900 2400 1800
+Wire Wire Line
+	2200 1500 2200 1400
+Wire Wire Line
+	2200 1400 1600 1400
+Wire Wire Line
+	1600 1300 2400 1300
+Wire Wire Line
+	2400 1300 2400 1500
 $EndSCHEMATC

Commit message: Hmmm
Connections:
- wire segments 192 -> 196
- no-connect marks 0 -> 1
Other:
- moved on the sheet: C1, C10, C11, C2, C3, C4, C5, C6, C8, C9, D1, J5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

Commit message: Hmmm
Parts:
- removed J4: ~, Connector_PinHeader_2.54mm:PinHeader_2x03_P2.54mm_Vertical, symbol Connector_Generic:Conn_02x03_Odd_Even
- removed U1: AMS1117-3.3, Package_TO_SOT_SMD:SOT-223-3_TabPin2, symbol Regulator_Linear:AMS1117-3.3
- added C12: 100nF, Capacitor_SMD:C_0402_1005Metric, symbol Device:C
- added JP1: ~, Jumper:SolderJumper-3_P1.3mm_Open_Pad1.0x1.5mm, symbol Jumper:SolderJumper_3_Open
- added R2: 10k, Resistor_SMD:R_0402_1005Metric, symbol Device:R
- added SW2: ~, Button_Switch_SMD:SW_SPST_TL3342, symbol Switch:SW_Push
- added U1: XC6206P332MR, Package_TO_SOT_SMD:SOT-23, symbol Regulator_Linear:XC6206PxxxMR
- SW1: value SW_Push -> ~
Connections:
- wire segments 196 -> 195
Other:
- moved on the sheet: D2, D3, R4, R5

Commit message: Almost ready
Parts:
- removed R2, R3: 10k, Resistor_SMD:R_0402_1005Metric, symbol Device:R
- Y1: LCSC (none) -> C115962
Connections:
- wire segments 195 -> 191
Other:
- note added: "Internal pull-up"
- moved on the sheet: C12, C7, SW1, SW2
Changed lines of the file:
@@
 L Switch:SW_Push SW1
 U 1 1 5F055544
-P 3300 6800
-F 0 "SW1" H 3200 6900 50  0000 C CNN
-F 1 "~" H 3500 6900 50  0000 C CNN
-F 2 "Button_Switch_SMD:SW_SPST_TL3342" H 3300 7000 50  0001 C CNN
-F 3 "https://datasheet.lcsc.com/szlcsc/1901111503_XKB-Enterprise-TS-1187A-B-A-B_C318884.pdf" H 3300 7000 50  0001 C CNN
-F 4 "C318884" H 3300 6800 50  0001 C CNN "LCSC"
-	1    3300 6800
+P 2600 6800
+F 0 "SW1" H 2500 6900 50  0000 C CNN
+F 1 "~" H 2800 6900 50  0000 C CNN
+F 2 "Button_Switch_SMD:SW_SPST_TL3342" H 2600 7000 50  0001 C CNN
+F 3 "https://datasheet.lcsc.com/szlcsc/1901111503_XKB-Enterprise-TS-1187A-B-A-B_C318884.pdf" H 2600 7000 50  0001 C CNN
+F 4 "C318884" H 2600 6800 50  0001 C CNN "LCSC"
+	1    2600 6800
 	0    -1   -1   0
 $EndComp
@@
 L power:GND #PWR0119
 U 1 1 5F055552
-P 3550 7150
-F 0 "#PWR0119" H 3550 6900 50  0001 C CNN
-F 1 "GND" H 3555 6977 50  0000 C CNN
-F 2 "" H 3550 7150 50  0001 C CNN
-F 3 "" H 3550 7150 50  0001 C CNN
-	1    3550 7150
+P 2850 7150
+F 0 "#PWR0119" H 2850 6900 50  0001 C CNN
+F 1 "GND" H 2855 6977 50  0000 C CNN
+F 2 "" H 2850 7150 50  0001 C CNN
+F 3 "" H 2850 7150 50  0001 C CNN
+	1    2850 7150
 	1    0    0    -1
 $EndComp
@@
 L Device:C C7
 U 1 1 5F066105
-P 3550 6800
-F 0 "C7" H 3550 6900 50  0000 L CNN
-F 1 "100nF" H 3550 6700 50  0000 L CNN
-F 2 "Capacitor_SMD:C_0402_1005Metric" H 3588 6650 50  0001 C CNN
-F 3 "~" H 3550 6800 50  0001 C CNN
-F 4 "C1525" H 3550 6800 50  0001 C CNN "LCSC"
-	1    3550 6800
-	1    0    0    -1
-$EndComp
-$Comp
-L Device:R R3
-U 1 1 5F06F3A6
-P 3550 6350
-F 0 "R3" H 3620 6396 50  0000 L CNN
-F 1 "10k" H 3620 6305 50  0000 L CNN
-F 2 "Resistor_SMD:R_0402_1005Metric" V 3480 6350 50  0001 C CNN
-F 3 "~" H 3550 6350 50  0001 C CNN
-F 4 "C25744" H 3550 6350 50  0001 C CNN "LCSC"
-	1    3550 6350
-	1    0    0    -1
-$EndComp
-$Comp
-L power:+3.3V #PWR0120
-U 1 1 5F0864E0
-P 3550 6100
-F 0 "#PWR0120" H 3550 5950 50  0001 C CNN
-F 1 "+3.3V" H 3565 6273 50  0000 C CNN
-F 2 "" H 3550 6100 50  0001 C CNN
-F 3 "" H 3550 6100 50  0001 C CNN
-	1    3550 6100
-	1    0    0    -1
-$EndComp
-Wire Wire Line
-	3550 6100 3550 6200
-Wire Wire Line
-	3550 6500 3550 6600
-Wire Wire Line
-	3300 6600 3550 6600
-Connection ~ 3550 6600
-Wire Wire Line
-	3550 6600 3550 6650
-Wire Wire Line
-	3300 7000 3300 7050
-Wire Wire Line
-	3300 7050 3550 7050
-Wire Wire Line
-	3550 7050 3550 6950
-Wire Wire Line
-	3550 7150 3550 7050
-Connection ~ 3550 7050
-Text GLabel 3750 6600 2    50   Input ~ 0
+P 2850 6800
+F 0 "C7" H 2850 6900 50  0000 L CNN
+F 1 "100nF" H 2850 6700 50  0000 L CNN
+F 2 "Capacitor_SMD:C_0402_1005Metric" H 2888 6650 50  0001 C CNN
+F 3 "~" H 2850 6800 50  0001 C CNN
+F 4 "C1525" H 2850 6800 50  0001 C CNN "LCSC"
+	1    2850 6800
+	1    0    0    -1
+$EndComp
+Wire Wire Line
+	2600 6600 2850 6600
+Connection ~ 2850 6600
+Wire Wire Line
+	2850 6600 2850 6650
+Wire Wire Line
+	2600 7000 2600 7050
+Wire Wire Line
+	2600 7050 2850 7050
+Wire Wire Line
+	2850 7050 2850 6950
+Wire Wire Line
+	2850 7150 2850 7050
+Connection ~ 2850 7050
+Text GLabel 3050 6600 2    50   Input ~ 0
 RST
 Wire Wire Line
-	3750 6600 3550 6600
+	3050 6600 2850 6600
 Text GLabel 6850 2300 0    50   Input ~ 0
 RST
@@
 F 2 "Crystal:Crystal_SMD_Abracon_ABM3-2Pin_5.0x3.2mm" H 4500 2900 50  0001 C CNN
 F 3 "~" H 4500 2900 50  0001 C CNN
+F 4 "C115962" H 4500 2900 50  0001 C CNN "LCSC"
 	1    4500 2900
 	1    0    0    -1
@@
 L Switch:SW_Push SW2
 U 1 1 5EFDDDE0
-P 4150 6350
-F 0 "SW2" H 4050 6450 50  0000 C CNN
-F 1 "~" H 4350 6450 50  0000 C CNN
-F 2 "Button_Switch_SMD:SW_SPST_TL3342" H 4150 6550 50  0001 C CNN
-F 3 "https://datasheet.lcsc.com/szlcsc/1901111503_XKB-Enterprise-TS-1187A-B-A-B_C318884.pdf" H 4150 6550 50  0001 C CNN
-F 4 "C318884" H 4150 6350 50  0001 C CNN "LCSC"
-	1    4150 6350
+P 3450 6800
+F 0 "SW2" H 3350 6900 50  0000 C CNN
+F 1 "~" H 3650 6900 50  0000 C CNN
+F 2 "Button_Switch_SMD:SW_SPST_TL3342" H 3450 7000 50  0001 C CNN
+F 3 "https://datasheet.lcsc.com/szlcsc/1901111503_XKB-Enterprise-TS-1187A-B-A-B_C318884.pdf" H 3450 7000 50  0001 C CNN
+F 4 "C318884" H 3450 6800 50  0001 C CNN "LCSC"
+	1    3450 6800
 	0    -1   -1   0
-$EndComp
-$Comp
-L Device:R R2
-U 1 1 5EFDE68B
-P 4350 6850
-F 0 "R2" H 4420 6896 50  0000 L CNN
-F 1 "10k" H 4420 6805 50  0000 L CNN
-F 2 "Resistor_SMD:R_0402_1005Metric" V 4280 6850 50  0001 C CNN
-F 3 "~" H 4350 6850 50  0001 C CNN
-F 4 "C25744" H 4350 6850 50  0001 C CNN "LCSC"
-	1    4350 6850
-	1    0    0    -1
 $EndComp
 $Comp
 L Device:C C12
 U 1 1 5EFDEFAE
-P 4350 6350
-F 0 "C12" H 4350 6450 50  0000 L CNN
-F 1 "100nF" H 4350 6250 50  0000 L CNN
-F 2 "Capacitor_SMD:C_0402_1005Metric" H 4388 6200 50  0001 C CNN
-F 3 "~" H 4350 6350 50  0001 C CNN
-F 4 "C1525" H 4350 6350 50  0001 C CNN "LCSC"
-	1    4350 6350
+P 3650 6800
+F 0 "C12" H 3650 6900 50  0000 L CNN
+F 1 "100nF" H 3650 6700 50  0000 L CNN
+F 2 "Capacitor_SMD:C_0402_1005Metric" H 3688 6650 50  0001 C CNN
+F 3 "~" H 3650 6800 50  0001 C CNN
+F 4 "C1525" H 3650 6800 50  0001 C CNN "LCSC"
+	1    3650 6800
 	1    0    0    -1
 $EndComp
@@
 L power:+3.3V #PWR0113
 U 1 1 5EFDFFB8
-P 4350 6100
-F 0 "#PWR0113" H 4350 5950 50  0001 C CNN
-F 1 "+3.3V" H 4365 6273 50  0000 C CNN
-F 2 "" H 4350 6100 50  0001 C CNN
-F 3 "" H 4350 6100 50  0001 C CNN
-	1    4350 6100
-	1    0    0    -1
-$EndComp
-$Comp
-L power:GND #PWR0114
-U 1 1 5EFE06DC
-P 4350 7150
-F 0 "#PWR0114" H 4350 6900 50  0001 C CNN
-F 1 "GND" H 4355 6977 50  0000 C CNN
-F 2 "" H 4350 7150 50  0001 C CNN
-F 3 "" H 4350 7150 50  0001 C CNN
-	1    4350 7150
-	1    0    0    -1
-$EndComp
-Text GLabel 4450 6600 2    50   Input ~ 0
+P 3650 6550
+F 0 "#PWR0113" H 3650 6400 50  0001 C CNN
+F 1 "+3.3V" H 3665 6723 50  0000 C CNN
+F 2 "" H 3650 6550 50  0001 C CNN
+F 3 "" H 3650 6550 50  0001 C CNN
+	1    3650 6550
+	1    0    0    -1
+$EndComp
+Text GLabel 3750 7050 2    50   Input ~ 0
 BO0
 Wire Wire Line
-	4350 6100 4350 6150
-Wire Wire Line
-	4150 6150 4350 6150
-Connection ~ 4350 6150
-Wire Wire Line
-	4350 6150 4350 6200
-Wire Wire Line
-	4150 6550 4150 6600
-Wire Wire Line
-	4150 6600 4350 6600
-Wire Wire Line
-	4350 6500 4350 6600
-Connection ~ 4350 6600
-Wire Wire Line
-	4350 6600 4450 6600
-Wire Wire Line
-	4350 6700 4350 6600
-Wire Wire Line
-	4350 7000 4350 7150
+	3650 6550 3650 6600
+Wire Wire Line
+	3450 6600 3650 6600
+Connection ~ 3650 6600
+Wire Wire Line
+	3650 6600 3650 6650
+Wire Wire Line
+	3450 7000 3450 7050
+Wire Wire Line
+	3450 7050 3650 7050
+Wire Wire Line
+	3650 6950 3650 7050
+Connection ~ 3650 7050
+Wire Wire Line
+	3650 7050 3750 7050
 $Comp
 L Jumper:SolderJumper_3_Open JP1
@@
 	1    0    0    -1
 $EndComp
+Text Notes 2600 6500 0    50   ~ 0
+Internal pull-up
 $EndSCHEMATC

Commit message: Hmm
Parts:
- added R1, R2: 22R, Resistor_SMD:R_0402_1005Metric, symbol Device:R
- added R3: 1.5k, Resistor_SMD:R_0402_1005Metric, symbol Device:R
- U2: value STM32F103C8Tx -> STM32F103C8T6
- renumbered C6 to C10, C10 to C11, C11 to C12, C7 to C3, C12 to C4, C8 to C5, C3 to C6, C9 to C7, C4 to C8, C5 to C9, J5 to J4, R6 to R4, R1 to R5, R4 to R6, R5 to R7
Connections:
- net labels added: +5V
- wire segments 191 -> 199
Other:
- note added: "Decoupling"
- note added: "Power Regulation"
- note added: "USB C Connection"
- moved on the sheet: C1, C10, C11, C12, C2, C5, C6, C7, C8, C9, D1, R4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

Commit message: Hmmm
Parts:
- removed JP1: ~, Jumper:SolderJumper-3_P1.3mm_Open_Pad1.0x1.5mm, symbol Jumper:SolderJumper_3_Open
Connections:
- net labels added: B2
- net labels removed: BO1
- wire segments 199 -> 197
Other:
- note added: "NOTICE! Headers are mostly but NOT\n100 % compatible with the blue/black pill."
- moved on the sheet: C11, C12, C3, C4, C5, C7, D2, D3, J3, J4, R6, R7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
