File: stm32devmini/stm32devmini.sch (KiCad schematic (older format))
At the start: 32 parts, among them J1 USB_C_Receptacle_USB2.0, U1 XC6206P332MR, U2 STM32F103C8T6, Y1 8M, Y2 32.768k

Commit message: stdm rev a
Connections:
- wire segments 197 -> 202
- no-connect marks 1 -> 5
Other:
- moved on the sheet: D1
Changed lines of the file:
@@
 L Device:D_Schottky D1
 U 1 1 5EF50EEB
-P 3450 2950
-F 0 "D1" H 3450 2825 50  0000 C CNN
-F 1 "~" H 3450 2824 50  0000 C CNN
-F 2 "Diode_SMD:D_SOD-123" H 3450 2950 50  0001 C CNN
-F 3 "~" H 3450 2950 50  0001 C CNN
-F 4 "C8598" H 3450 2950 50  0001 C CNN "LCSC"
-	1    3450 2950
+P 3050 2950
+F 0 "D1" H 3050 2825 50  0000 C CNN
+F 1 "~" H 3050 2824 50  0000 C CNN
+F 2 "Diode_SMD:D_SOD-123" H 3050 2950 50  0001 C CNN
+F 3 "~" H 3050 2950 50  0001 C CNN
+F 4 "C8598" H 3050 2950 50  0001 C CNN "LCSC"
+	1    3050 2950
 	-1   0    0    1
 $EndComp
@@
 $EndComp
 Wire Wire Line
-	1150 1650 1150 1450
+	1150 1650 1150 1550
 $Comp
 L power:GND #PWR08
@@
 $EndComp
 Wire Wire Line
-	1600 2950 3250 2950
+	1600 2950 1850 2950
 Wire Wire Line
 	3100 3650 3100 3750
@@
 L power:VBUS #PWR012
 U 1 1 5F008BB0
-P 3250 2850
-F 0 "#PWR012" H 3250 2700 50  0001 C CNN
-F 1 "VBUS" H 3265 3023 50  0000 C CNN
-F 2 "" H 3250 2850 50  0001 C CNN
-F 3 "" H 3250 2850 50  0001 C CNN
-	1    3250 2850
-	1    0    0    -1
-$EndComp
-Wire Wire Line
-	3600 2950 3700 2950
+P 2750 2850
+F 0 "#PWR012" H 2750 2700 50  0001 C CNN
+F 1 "VBUS" H 2765 3023 50  0000 C CNN
+F 2 "" H 2750 2850 50  0001 C CNN
+F 3 "" H 2750 2850 50  0001 C CNN
+	1    2750 2850
+	1    0    0    -1
+$EndComp
+Wire Wire Line
+	3200 2950 3350 2950
 Wire Wire Line
 	3700 2950 3700 2850
@@
 Connection ~ 2800 1100
 Wire Wire Line
-	3250 2850 3250 2950
-Connection ~ 3250 2950
-Wire Wire Line
-	3250 2950 3300 2950
+	2750 2850 2750 2950
+Connection ~ 2750 2950
+Wire Wire Line
+	2750 2950 2900 2950
 $Comp
 L Device:R R1
@@
 Text Notes 9450 6350 0    50   ~ 0
 NOTICE!  Headers are mostly but NOT\n100 % compatible with the blue/black pill.
+$Comp
+L power:PWR_FLAG #FLG0101
+U 1 1 5F1B7E76
+P 1850 2850
+F 0 "#FLG0101" H 1850 2925 50  0001 C CNN
+F 1 "PWR_FLAG" H 1850 3023 50  0000 C CNN
+F 2 "" H 1850 2850 50  0001 C CNN
+F 3 "~" H 1850 2850 50  0001 C CNN
+	1    1850 2850
+	1    0    0    -1
+$EndComp
+Wire Wire Line
+	1850 2850 1850 2950
+Connection ~ 1850 2950
+Wire Wire Line
+	1850 2950 2750 2950
+NoConn ~ 1600 4050
+NoConn ~ 1600 4150
+NoConn ~ 3800 4450
+$Comp
+L power:PWR_FLAG #FLG0102
+U 1 1 5F1F0DFA
+P 1150 1550
+F 0 "#FLG0102" H 1150 1625 50  0001 C CNN
+F 1 "PWR_FLAG" V 1150 1678 50  0000 L CNN
+F 2 "" H 1150 1550 50  0001 C CNN
+F 3 "~" H 1150 1550 50  0001 C CNN
+	1    1150 1550
+	0    1    1    0
+$EndComp
+Connection ~ 1150 1550
+Wire Wire Line
+	1150 1550 1150 1450
+NoConn ~ 3150 900
+$Comp
+L power:PWR_FLAG #FLG0103
+U 1 1 5F2349A8
+P 3350 2850
+F 0 "#FLG0103" H 3350 2925 50  0001 C CNN
+F 1 "PWR_FLAG" H 3350 3023 50  0000 C CNN
+F 2 "" H 3350 2850 50  0001 C CNN
+F 3 "~" H 3350 2850 50  0001 C CNN
+	1    3350 2850
+	1    0    0    -1
+$EndComp
+Wire Wire Line
+	3350 2850 3350 2950
+Connection ~ 3350 2950
+Wire Wire Line
+	3350 2950 3700 2950
 $EndSCHEMATC

Commit message: Hmmmmm
Parts:
- removed C4: 100nF, Capacitor_SMD:C_0402_1005Metric, symbol Device:C
- added R8: 1k, Resistor_SMD:R_0402_1005Metric, symbol Device:R
- added R9: NM, Resistor_SMD:R_0402_1005Metric, symbol Device:R
- R6: value 1k -> NM; LCSC C25905 -> (none)
- SW1, SW2: LCSC C318884 -> C318887
Connections:
- no-connect marks 5 -> 4
Other:
- moved on the sheet: C11, C12, C3, C5, C7, R6, SW1, SW2, U2, Y1, Y2

Commit message: Hmmmm
Other:
- note added: "LEDs"
- note added: "Pin Headers"
- note added: "Processor"
- note added: "Programming Header"
- note added: "Reset & Boot Mode"
- moved on the sheet: J2
Changed lines of the file:
@@
 L Connector_Generic:Conn_01x20 J2
 U 1 1 5EF5C946
-P 10750 1800
-F 0 "J2" H 10830 1746 50  0000 L CNN
-F 1 "~" H 10830 1701 50  0000 L CNN
-F 2 "Connector_PinHeader_2.54mm:PinHeader_1x20_P2.54mm_Vertical" H 10750 1800 50  0001 C CNN
-F 3 "~" H 10750 1800 50  0001 C CNN
-	1    10750 1800
+P 10750 2100
+F 0 "J2" H 10830 2046 50  0000 L CNN
+F 1 "~" H 10830 2001 50  0000 L CNN
+F 2 "Connector_PinHeader_2.54mm:PinHeader_1x20_P2.54mm_Vertical" H 10750 2100 50  0001 C CNN
+F 3 "~" H 10750 2100 50  0001 C CNN
+	1    10750 2100
 	1    0    0    -1
 $EndComp
@@
 Wire Wire Line
 	7600 4450 7700 4450
-Text GLabel 9900 1000 0    50   Input ~ 0
+Text GLabel 9900 1300 0    50   Input ~ 0
 C13
-Text GLabel 9900 1100 0    50   Input ~ 0
+Text GLabel 9900 1400 0    50   Input ~ 0
 C14
-Text GLabel 9900 1200 0    50   Input ~ 0
+Text GLabel 9900 1500 0    50   Input ~ 0
 C15
 Wire Wire Line
-	9900 1000 10550 1000
-Wire Wire Line
-	10550 1100 9900 1100
-Wire Wire Line
-	9900 1200 10550 1200
-Text GLabel 9900 1300 0    50   Input ~ 0
+	9900 1300 10550 1300
+Wire Wire Line
+	10550 1400 9900 1400
+Wire Wire Line
+	9900 1500 10550 1500
+Text GLabel 9900 1600 0    50   Input ~ 0
 A0
-Text GLabel 9900 1400 0    50   Input ~ 0
+Text GLabel 9900 1700 0    50   Input ~ 0
 A1
-Text GLabel 9900 1500 0    50   Input ~ 0
+Text GLabel 9900 1800 0    50   Input ~ 0
 A2
 Wire Wire Line
-	9900 1300 10550 1300
-Wire Wire Line
-	10550 1400 9900 1400
-Wire Wire Line
-	9900 1500 10550 1500
+	9900 1600 10550 1600
+Wire Wire Line
+	10550 1700 9900 1700
+Wire Wire Line
+	9900 1800 10550 1800
 Text GLabel 10050 3850 0    50   Input ~ 0
 B9
@@
 	10050 5450 10550 5450
 Wire Wire Line
-	9900 1600 10550 1600
-Text GLabel 9900 1600 0    50   Input ~ 0
+	9900 1900 10550 1900
+Text GLabel 9900 1900 0    50   Input ~ 0
 A3
-Text GLabel 9900 1700 0    50   Input ~ 0
+Text GLabel 9900 2000 0    50   Input ~ 0
 A4
-Text GLabel 9900 1800 0    50   Input ~ 0
+Text GLabel 9900 2100 0    50   Input ~ 0
 A5
-Text GLabel 9900 1900 0    50   Input ~ 0
+Text GLabel 9900 2200 0    50   Input ~ 0
 A6
-Text GLabel 9900 2000 0    50   Input ~ 0
+Text GLabel 9900 2300 0    50   Input ~ 0
 A7
 Wire Wire Line
-	9900 2000 10550 2000
-Wire Wire Line
-	10550 1900 9900 1900
-Wire Wire Line
-	9900 1800 10550 1800
-Wire Wire Line
-	10550 1700 9900 1700
-Text GLabel 9900 2100 0    50   Input ~ 0
+	9900 2300 10550 2300
+Wire Wire Line
+	10550 2200 9900 2200
+Wire Wire Line
+	9900 2100 10550 2100
+Wire Wire Line
+	10550 2000 9900 2000
+Text GLabel 9900 2400 0    50   Input ~ 0
 B0
-Text GLabel 9900 2200 0    50   Input ~ 0
+Text GLabel 9900 2500 0    50   Input ~ 0
 B1
-Text GLabel 9900 2400 0    50   Input ~ 0
+Text GLabel 9900 2700 0    50   Input ~ 0
 B10
-Text GLabel 9900 2500 0    50   Input ~ 0
+Text GLabel 9900 2800 0    50   Input ~ 0
 B11
 Wire Wire Line
-	9900 2100 10550 2100
-Wire Wire Line
-	10550 2200 9900 2200
-Wire Wire Line
-	9900 2300 10550 2300
-Wire Wire Line
 	9900 2400 10550 2400
+Wire Wire Line
+	10550 2500 9900 2500
+Wire Wire Line
+	9900 2600 10550 2600
+Wire Wire Line
+	9900 2700 10550 2700
 Text GLabel 2650 3650 2    50   Input ~ 0
 A12
@@
 	1700 3650 1600 3650
 Wire Wire Line
-	10450 900  10550 900
+	10450 1200 10550 1200
 $Comp
 L power:+3.3V #PWR031
 U 1 1 5EF5F475
-P 10000 800
-F 0 "#PWR031" H 10000 650 50  0001 C CNN
-F 1 "+3.3V" H 10015 973 50  0000 C CNN
-F 2 "" H 10000 800 50  0001 C CNN
-F 3 "" H 10000 800 50  0001 C CNN
-	1    10000 800
-	1    0    0    -1
-$EndComp
-Wire Wire Line
-	10000 2600 10550 2600
-Wire Wire Line
-	10000 800  10000 2600
-Wire Wire Line
-	9900 2500 10550 2500
+P 10000 1100
+F 0 "#PWR031" H 10000 950 50  0001 C CNN
+F 1 "+3.3V" H 10015 1273 50  0000 C CNN
+F 2 "" H 10000 1100 50  0001 C CNN
+F 3 "" H 10000 1100 50  0001 C CNN
+	1    10000 1100
+	1    0    0    -1
+$EndComp
+Wire Wire Line
+	10000 2900 10550 2900
+Wire Wire Line
+	10000 1100 10000 2900
+Wire Wire Line
+	9900 2800 10550 2800
 $Comp
 L power:GND #PWR034
 U 1 1 5EF9371A
-P 10450 2900
-F 0 "#PWR034" H 10450 2650 50  0001 C CNN
-F 1 "GND" H 10455 2727 50  0000 C CNN
-F 2 "" H 10450 2900 50  0001 C CNN
-F 3 "" H 10450 2900 50  0001 C CNN
-	1    10450 2900
-	1    0    0    -1
-$EndComp
-Wire Wire Line
-	10450 2900 10450 2800
-Wire Wire Line
-	10550 2800 10450 2800
+P 10450 3200
+F 0 "#PWR034" H 10450 2950 50  0001 C CNN
+F 1 "GND" H 10455 3027 50  0000 C CNN
+F 2 "" H 10450 3200 50  0001 C CNN
+F 3 "" H 10450 3200 50  0001 C CNN
+	1    10450 3200
+	1    0    0    -1
+$EndComp
+Wire Wire Line
+	10450 3200 10450 3100
+Wire Wire Line
+	10550 3100 10450 3100
 $Comp
 L Device:R R5
@@
 L power:+5V #PWR0101
 U 1 1 5F1B0776
-P 10200 800
-F 0 "#PWR0101" H 10200 650 50  0001 C CNN
-F 1 "+5V" H 10215 973 50  0000 C CNN
-F 2 "" H 10200 800 50  0001 C CNN
-F 3 "" H 10200 800 50  0001 C CNN
-	1    10200 800
+P 10200 1100
+F 0 "#PWR0101" H 10200 950 50  0001 C CNN
+F 1 "+5V" H 10215 1273 50  0000 C CNN
+F 2 "" H 10200 1100 50  0001 C CNN
+F 3 "" H 10200 1100 50  0001 C CNN
+	1    10200 1100
 	1    0    0    -1
 $EndComp
@@
 USB C Connection
 Wire Wire Line
-	10450 900  10450 2800
-Connection ~ 10450 2800
-Wire Wire Line
-	10550 2700 10200 2700
-Wire Wire Line
-	10200 2700 10200 800
+	10450 1200 10450 3100
+Connection ~ 10450 3100
+Wire Wire Line
+	10550 3000 10200 3000
+Wire Wire Line
+	10200 3000 10200 1100
 Wire Wire Line
 	10550 3550 10450 3550
@@
 Text GLabel 6800 2850 0    50   Input ~ 0
 B2
-Text GLabel 9900 2300 0    50   Input ~ 0
+Text GLabel 9900 2600 0    50   Input ~ 0
 B2
-Text Notes 9450 6350 0    50   ~ 0
+Text Notes 9350 6350 0    50   ~ 0
 NOTICE!  Headers are mostly but NOT\n100 % compatible with the blue/black pill.
 $Comp
@@
 Wire Wire Line
 	2200 6450 2200 6550
+Wire Notes Line
+	9300 700  9300 6400
+Wire Notes Line
+	9300 6400 11000 6400
+Wire Notes Line
+	11000 6400 11000 700
+Wire Notes Line
+	11000 700  9300 700
+Text Notes 4350 650  0    50   ~ 0
+Processor
+Text Notes 9300 650  0    50   ~ 0
+Pin Headers
+Wire Notes Line
+	550  7450 2700 7450
+Wire Notes Line
+	2700 7450 2700 5450
+Wire Notes Line
+	2700 5450 550  5450
+Wire Notes Line
+	550  5450 550  7450
+Text Notes 550  5400 0    50   ~ 0
+Reset & Boot Mode
+Wire Notes Line
+	3050 7450 4550 7450
+Wire Notes Line
+	4550 7450 4550 5450
+Wire Notes Line
+	4550 5450 3050 5450
+Wire Notes Line
+	3050 5450 3050 7450
+Text Notes 3050 5400 0    50   ~ 0
+LEDs
+Wire Notes Line
+	4850 7450 6250 7450
+Wire Notes Line
+	6250 7450 6250 5450
+Wire Notes Line
+	6250 5450 4850 5450
+Wire Notes Line
+	4850 5450 4850 7450
+Text Notes 4850 5400 0    50   ~ 0
+Programming Header
 $EndSCHEMATC
