File: pcb/stm32dev.kicad_pcb (KiCad board)
At the start: 2 copper layers, 39.4 x 26.7 mm, 24 parts, among them J1 USB_B_Micro, J2 Micro_SD_Card_Det, U1 AMS1117-3.3, U2 STM32F405RGTx, Y1 16 MHz

Commit message: Hmmm
Routing:
- net VCC: track 84.7 -> 84.0 mm
- net RGB: track 17.6 -> 16.9 mm

Commit message: Hmmm
Routing:
- net EN: track 19.8 -> 19.5 mm, vias 0 -> 2
- net VCC: track 84.0 -> 84.2 mm, vias 9 -> 8
Other:
- board text added: "STM32F504 Dev Board rev. a"
- board text removed: "STM32F504 Dev Board Rev. 1"

Commit message: Hmmm
Parts:
- moved C11 1.80 mm to (141.6, 92.7)
- moved C1 0.64 mm to (171.4, 106.0)
Routing:
- net PA0: track 28.1 -> 15.4 mm
- net VBUS: track 28.5 -> 27.8 mm
- net GND: vias 11 -> 10
Other:
- board text added: "AI0"
- board text added: "AI1"
- board text added: "AO0"
- board text added: "AO1"
- board text added: "C1RX"
- board text added: "C1TX"
- board text added: "C2RX"
- board text added: "C2TX"
- board text added: "JCLK"
- board text added: "JDI"
- board text added: "JDO"
- board text added: "JLCJLCJLCJLC"
- board text added: "JMS"
- board text added: "JRST"
- board text added: "MISO"
- board text added: "MOSI"
- board text added: "SCK"
- board text added: "SCL"
- board text added: "SDA"
- board text added: "U2RX"
- board text added: "U2TX"
- board text added: "VB"

Commit message: Hmmm
Parts:
- added J7: USB_C_Receptacle_USB2.0, Connector_USB:USB_C_Receptacle_HRO_TYPE-C-31-M-12, F.Cu at (182.5, 97.5)

Commit message: Hmmmm
Parts:
- removed C11, C9: 100nF, Capacitor_SMD:C_0402_1005Metric
- removed C3: 10uF, Capacitor_SMD:C_0805_2012Metric
- removed J7: USB_C_Receptacle_USB2.0, Connector_USB:USB_C_Receptacle_HRO_TYPE-C-31-M-12
- C10, C12, C13, C6: footprint Capacitor_SMD:C_0603_1608Metric -> Capacitor_SMD:C_0402_1005Metric

Commit message: hmmmm
Parts:
- added C3: 100nF, Capacitor_SMD:C_0402_1005Metric, F.Cu at (132.6, 89.5)
- added C9: 100nF, Capacitor_SMD:C_0402_1005Metric, F.Cu at (132.7, 100.3)
- added R1: 10k, Resistor_SMD:R_0402_1005Metric, F.Cu at (132.2, 91.4)
- added R2: 22R, Resistor_SMD:R_0402_1005Metric, F.Cu at (132.1, 93.5)
- added R3: 22R, Resistor_SMD:R_0402_1005Metric, F.Cu at (131.4, 95.9)
- added R4: 10k, Resistor_SMD:R_0402_1005Metric, F.Cu at (133.3, 103.5)
- added SW1: ~, Button_Switch_SMD:SW_SPST_TL3342, F.Cu at (127.0, 91.4)
- added SW2: ~, Button_Switch_SMD:SW_SPST_TL3342, F.Cu at (127.0, 104.1)
- J3, J4: footprint Connector_PinHeader_2.54mm:PinHeader_1x15_P2.54mm_Vertical -> Connector_PinHeader_2.54mm:PinHeader_1x20_P2.54mm_Vertical
- J5: footprint Connector_PinHeader_2.54mm:PinHeader_2x03_P2.54mm_Vertical -> Connector_PinHeader_2.54mm:PinHeader_1x06_P2.54mm_Vertical
- moved D2 39.2 mm to (127.0, 97.8), turned to 0 degrees
- moved J5 20.4 mm to (137.8, 91.4)
- moved J2 12.7 mm to (129.5, 97.8)
- moved J3 12.7 mm to (124.5, 109.2)
- moved J4 12.7 mm to (124.5, 86.4)
- moved C13 4.45 mm to (160.0, 90.2)
- moved C10 3.81 mm to (142.9, 99.1)
- moved C6 3.81 mm to (142.9, 92.7)
- moved Y1 3.81 mm to (142.9, 95.9)
- moved C7 3.81 mm to (158.3, 92.7)
- moved U2 3.60 mm to (151.8, 97.8)
- moved C12 2.54 mm to (156.8, 104.8)
- moved C8 2.54 mm to (157.5, 102.9)
- moved J1 0.64 mm to (171.4, 97.8)
Connections:
- J1 pad 2: DM -> Net-(J1-Pad2)
- J1 pad 3: DP -> Net-(J1-Pad3)
- J3 pad 1: GND -> Net-(J3-Pad1)
- J3 pad 10: PA5_AO1 -> PA3_U2_RX
- J3 pad 11: PA6_AI0 -> PA4_AO0
- J3 pad 12: PA7_AI1 -> PA5_AO1
- J3 pad 13: VCC -> PA6_AI0
- J3 pad 14: VBUS -> PA7_AI1
- J3 pad 15: GND -> VCC
- J3 pad 2: PC2_MISO -> Net-(J3-Pad2)
- J3 pad 3: PC3_MOSI -> GND
- J3 pad 4: PB10_SCK -> PC2_MISO
- J3 pad 5: PA0 -> PC3_MOSI
- J3 pad 6: PA1 -> PB10_SCK
- J3 pad 7: PA2_U2_TX -> PA0
- J3 pad 8: PA3_U2_RX -> PA1
- J3 pad 9: PA4_AO0 -> PA2_U2_TX
- J4 pad 1: GND -> Net-(J4-Pad1)
- J4 pad 10: PA13_JMS -> PB3_JDO
- J4 pad 11: PC7 -> PA15_JDI
- J4 pad 12: PC6 -> PA14_JCLK
- J4 pad 13: PB13_CAN2_TX -> PA13_JMS
- J4 pad 14: PB12_CAN2_RX -> PC7
- J4 pad 15: GND -> PC6
- J4 pad 2: PB9_CAN1_RX -> Net-(J4-Pad2)
- J4 pad 3: PB8_CAN1_TX -> Net-(J4-Pad3)
- J4 pad 4: PB7_SDA -> GND
- J4 pad 5: PB6_SCL -> PB9_CAN1_RX
- J4 pad 6: PB4_JRST -> PB8_CAN1_TX
- J4 pad 7: PB3_JDO -> PB7_SDA
- J4 pad 8: PA15_JDI -> PB6_SCL
- J4 pad 9: PA14_JCLK -> PB4_JRST
- U2 pad 60: 0 -> BO0
- U2 pad 7: EN -> NRST
Routing:
- net VCC: track 84.5 -> 0.00 mm, vias 8 -> 0
- net VBUS: track 27.8 -> 0.00 mm, vias 2 -> 0
- net PB12_CAN2_RX: track 24.0 -> 0.00 mm, vias 1 -> 0
- net PB13_CAN2_TX: track 22.2 -> 0.00 mm, vias 1 -> 0
- net PC6: track 20.9 -> 0.00 mm
- net PA7_AI1: track 20.6 -> 0.00 mm
- net EN: track 19.5 -> 0.00 mm, vias 2 -> 0
- net SD_D1: track 19.1 -> 0.00 mm, vias 1 -> 0
- net PC7: track 19.0 -> 0.00 mm
- net PA6_AI0: track 18.5 -> 0.00 mm
- net SD_CLK: track 18.1 -> 0.00 mm, vias 1 -> 0
- net SD_D3: track 18.1 -> 0.00 mm, vias 1 -> 0
- net PA3_U2_RX: track 17.9 -> 0.00 mm
- net SD_D0: track 17.8 -> 0.00 mm, vias 1 -> 0
- net PA2_U2_TX: track 17.6 -> 0.00 mm
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Other:
- board size 39.4 x 26.7 mm -> 52.1 x 26.7 mm
- board text added: "STM32F504 Dev Board rev. b"
- board text removed: "STM32F504 Dev Board rev. a"

Commit message: Hmmmmm
Parts:
- removed R1, R4: 10k, Resistor_SMD:R_0402_1005Metric
- added C11: 1uF, Capacitor_SMD:C_0402_1005Metric, F.Cu at (156.8, 106.0)
- C10, C6: value 22pF -> 20pF
- U1: value AMS1117-3.3 -> XC6206P332MR; footprint Package_TO_SOT_SMD:SOT-223-3_TabPin2 -> Package_TO_SOT_SMD:SOT-23
- Y1: value 16 MHz -> 8 MHz; footprint Crystal:Crystal_SMD_3225-4Pin_3.2x2.5mm -> Crystal:Crystal_SMD_Abracon_ABM3-2Pin_5.0x3.2mm
- moved R3 36.3 mm to (167.6, 98.4)
- moved R2 35.7 mm to (167.6, 97.2)
- moved SW1 12.7 mm to (127.0, 104.1), turned to 180 degrees
- moved SW2 12.7 mm to (127.0, 91.4)
- moved C2 3.24 mm to (163.2, 104.8)
- moved U1 2.84 mm to (166.4, 104.8), turned to 0 degrees
- moved C10 0.90 mm to (142.2, 99.7)
- moved C6 0.90 mm to (142.2, 92.1)
- moved Y1 0.63 mm to (142.2, 95.9)
Connections:
- net Net-(U2-Pad26) renamed PB0
- net Net-(U2-Pad27) renamed PB1
- net Net-(U2-Pad28) renamed PB2
- net Net-(U2-Pad30) renamed PB11
- net Net-(U2-Pad41) renamed PA8
- C2 pad 1: VCC -> +3V3
- C4 pad 1: VCC -> +3V3
- C5 pad 1: VCC -> +3V3
- C7 pad 1: VCC -> +3V3
- C8 pad 1: VCC -> +3V3
- D2 pad 1: VCC -> +3V3
- J2 pad 4: VCC -> +3V3
- J3 pad 1: Net-(J3-Pad1) -> GND
- J3 pad 15: VCC -> Net-(J3-Pad15)
- J3 pad 16: VBUS -> Net-(J3-Pad16)
- J3 pad 17: GND -> Net-(J3-Pad17)
- J3 pad 18: Net-(J3-Pad18) -> +3V3
- J3 pad 19: Net-(J3-Pad19) -> VBUS
- J3 pad 20: Net-(J3-Pad20) -> GND
- J3 pad 3: GND -> Net-(J3-Pad3)
- J4 pad 1: Net-(J4-Pad1) -> GND
- J4 pad 18: GND -> Net-(J4-Pad18)
- J4 pad 20: Net-(J4-Pad20) -> GND
- J4 pad 4: GND -> Net-(J4-Pad4)
- R2 pad 1: DP -> PA12
- R3 pad 1: DM -> PA11
- SW2 pad 1: VCC -> +3V3
- U1 pad 2: VCC -> +3V3
- U2 pad 1: VCC -> +3V3
- U2 pad 13: VCC -> +3V3
- U2 pad 16: PA2_U2_TX -> PA2
- U2 pad 17: PA3_U2_RX -> PA3
- U2 pad 19: VCC -> +3V3
- U2 pad 20: PA4_AO0 -> PA4
- U2 pad 21: PA5_AO1 -> PA5
- U2 pad 22: PA6_AI0 -> PA6
- U2 pad 23: PA7_AI1 -> PA7
- U2 pad 29: PB10_SCK -> PB10
- U2 pad 32: VCC -> +3V3
- U2 pad 33: PB12_CAN2_RX -> PB12
- U2 pad 34: PB13_CAN2_TX -> PB13
- U2 pad 35: DM -> PB14
- U2 pad 36: DP -> PB15
- U2 pad 42: RXD -> PA9
- U2 pad 43: TXD -> PA10
- U2 pad 44: Net-(U2-Pad44) -> PA11
- U2 pad 45: RGB -> PA12
- U2 pad 46: PA13_JMS -> PA13
- U2 pad 48: VCC -> +3V3
- U2 pad 49: PA14_JCLK -> PA14
- U2 pad 50: PA15_JDI -> PA15
- U2 pad 55: PB3_JDO -> PB3
- U2 pad 56: PB4_JRST -> PB4
- U2 pad 58: PB6_SCL -> PB6
- U2 pad 59: PB7_SDA -> PB7
- U2 pad 61: PB8_CAN1_TX -> PB8
- U2 pad 62: PB9_CAN1_RX -> PB9
- U2 pad 64: VCC -> +3V3
- Y1 pad 2: GND -> Net-(C10-Pad1)
Routing:
- removed copper zone on B.Cu, net VCC
- removed copper zone on F.Cu, net VCC

Commit message: Hmmmm
Parts:
- removed C9: 100nF, Capacitor_SMD:C_0402_1005Metric
- added D4: ~, Diode_SMD:D_SOD-123, F.Cu at (149.8, 75.0)
- added D5: BLUE, LED_SMD:LED_0603_1608Metric, F.Cu at (154.7, 74.7)
- added R1: NM, Resistor_SMD:R_0402_1005Metric, F.Cu at (157.0, 77.0)
- added R4: 22R, Resistor_SMD:R_0402_1005Metric, F.Cu at (172.5, 66.5)
- added R5: 1.5k, Resistor_SMD:R_0402_1005Metric, F.Cu at (169.6, 70.5)
- added R6: 1k, Resistor_SMD:R_0402_1005Metric, F.Cu at (172.5, 68.5)
- added R7: 5.1k, Resistor_SMD:R_0402_1005Metric, F.Cu at (169.6, 72.5)
- added R8: 1k, Resistor_SMD:R_0402_1005Metric, F.Cu at (172.5, 70.5)
- added R9: 5.1k, Resistor_SMD:R_0402_1005Metric, F.Cu at (169.6, 74.5)
- D1: value ~ -> YEL; footprint Diode_SMD:D_SOD-123 -> LED_SMD:LED_0603_1608Metric
- J1: value USB_B_Micro -> USB_C_Receptacle_USB2.0; footprint Connector_USB:USB_Micro-B_Molex-105017-0001 -> Connector_USB:USB_C_Receptacle_HRO_TYPE-C-31-M-12; moved to B.Cu
- J5: footprint Connector_PinHeader_2.54mm:PinHeader_1x06_P2.54mm_Vertical -> Connector_PinHeader_2.54mm:PinHeader_1x06_P2.54mm_Horizontal
- R2: value 22R -> NM
- moved D1 39.5 mm to (170.2, 64.2)
- moved R2 30.7 mm to (169.6, 66.5)
- moved R3 30.0 mm to (169.6, 68.5)
- moved C3 24.9 mm to (154.1, 77.0)
- moved J5 18.9 mm to (123.8, 104.1), turned to 180 degrees
- moved SW1 13.3 mm to (130.8, 91.4), turned to 0 degrees
- moved SW2 13.3 mm to (130.8, 104.1)
- moved C10 4.07 mm to (139.7, 102.9)
- moved C6 4.07 mm to (139.7, 95.2)
- moved Y1 4.07 mm to (139.7, 99.1)
- moved D2 3.81 mm to (130.8, 97.8)
- moved J2 3.18 mm to (132.7, 97.8), turned to 270 degrees
- moved C5 2.62 mm to (147.3, 104.8)
- moved J3 1.27 mm to (124.5, 108.0)
- moved J4 1.27 mm to (124.5, 87.6)
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Connections:
- C1 pad 1: VBUS -> +5V
- D1 pad 1: VBUS -> Net-(D1-Pad1)
- D1 pad 2: Net-(D1-Pad2) -> +3V3
- R2 pad 1: PA12 -> BO0
- R2 pad 2: Net-(J1-Pad3) -> GND
- R3 pad 1: PA11 -> Net-(J1-PadA7)
- R3 pad 2: Net-(J1-Pad2) -> PA11
- SW2 pad 1: +3V3 -> BO0
- SW2 pad 2: BO0 -> +3V3
- U1 pad 3: VBUS -> +5V
Routing:
- net Net-(D3-Pad2): vias 1 -> 0
- net GND: vias 0 -> 1
