File: pcb/stm32dev.kicad_pcb (KiCad board)
At the start: 2 copper layers, 52.1 x 30.5 mm, 36 parts, among them J1 USB_C_Receptacle_USB2.0, J3 Micro_SD_Card_Det, U1 XC6206P332MR, U2 STM32F405RGTx, Y1 8 MHz

Commit message: Few tweaks towards rev c
Other:
- board text added: "STM32F405 Dev Board rev. c"
- board text removed: "STM32F504 Dev Board rev. b"
Changed lines of the file:
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@@
   (title_block
     (title "STM32 Dev Board")
-    (rev b)
+    (rev c)
     (company "Lars Boegild Thomsen")
     (comment 1 lbthomsen@gmail.com)
@@
   )
   (setup
-    (last_trace_width 0.2286)
+    (last_trace_width 0.1524)
     (user_trace_width 0.1524)
     (user_trace_width 0.2286)
@@
     (effects (font (size 0.8 0.8) (thickness 0.15)) (justify left mirror))
   )
-  (gr_text "STM32F504 Dev Board\nrev. b" (at 164.465 97.155) (layer B.SilkS)
+  (gr_text "STM32F405 Dev Board\nrev. c" (at 164.465 97.155) (layer B.SilkS)
     (effects (font (size 0.8 0.8) (thickness 0.15)) (justify left mirror))
   )

Commit message: Hmmmmm
Parts:
- removed R4: 1.5k, Resistor_SMD:R_0402_1005Metric
- D1: value WS2812B -> WS2812B-Mini; footprint LED_SMD:LED_WS2812B_PLCC4_5.0x5.0mm_P3.2mm -> stm32dev:LED_WS2812B_MINI_3.5x3.5mm_P1.9mm
- J1: value USB_C_Receptacle_USB2.0 -> ~
- R6, R9: value 1k -> 220
- SW1, SW2: footprint Button_Switch_SMD:SW_SPST_TL3342 -> stm32dev:TS-1088R-02526
- Y1: value 8 MHz -> 16 MHz; footprint Crystal:Crystal_SMD_Abracon_ABM3-2Pin_5.0x3.2mm -> Crystal:Crystal_SMD_3225-4Pin_3.2x2.5mm
Connections:
- R7 pad 1: Net-(J1-PadB5) -> Net-(J1-PadA5)
- R7 pad 2: GND -> UCC
- R8 pad 1: Net-(J1-PadA5) -> Net-(J1-PadB5)
- R8 pad 2: GND -> UCC
- U2 pad 3: Net-(U2-Pad3) -> UCC
- Y1 pad 2: Net-(C11-Pad1) -> GND

Commit message: Hmmm
Parts:
- J1: footprint Connector_USB:USB_C_Receptacle_HRO_TYPE-C-31-M-12 -> stm32dev:USB_C_Receptacle_HRO_TYPE-C-31-M-12; moved to F.Cu
- moved D1 28.0 mm to (160.0, 91.4), turned to 180 degrees
- moved R7 8.35 mm to (163.8, 99.7), turned to 180 degrees
- moved R2 8.25 mm to (163.8, 97.2), turned to 180 degrees
- moved R3 8.25 mm to (163.8, 98.4), turned to 180 degrees
- moved R8 8.25 mm to (163.8, 95.9), turned to 180 degrees
- moved C1 7.62 mm to (163.8, 104.1), turned to 270 degrees
- moved C3 6.48 mm to (157.5, 104.1), turned to 270 degrees
- moved D2 6.35 mm to (167.6, 104.8), turned to 0 degrees
- moved U1 5.46 mm to (160.7, 104.1), turned to 270 degrees
- moved D4 5.43 mm to (167.6, 90.8)
- moved R9 5.43 mm to (165.1, 90.8)
- moved J1 1.42 mm to (170.8, 97.8), turned to 90 degrees
Routing:
- net +3V3: track 202.7 -> 0.00 mm, vias 6 -> 4
- net PA12: track 46.0 -> 0.00 mm, vias 2 -> 0
- net PA11: track 43.5 -> 0.00 mm, vias 2 -> 0
- net SWDIO: track 37.1 -> 0.00 mm
- net SWCLK: track 33.8 -> 0.00 mm, vias 2 -> 1
- net PC6: track 32.4 -> 0.00 mm, vias 2 -> 0
- net SD_DET: track 31.1 -> 0.00 mm
- net PC13: track 30.2 -> 0.00 mm, vias 2 -> 1
- net SD_D1: track 29.3 -> 0.00 mm
- net SWO: track 26.4 -> 0.00 mm
- net PB9: track 26.1 -> 0.00 mm
- net PB10: track 25.8 -> 0.00 mm
- net PC0: track 25.2 -> 0.00 mm
- net PA10: track 25.1 -> 0.00 mm, vias 1 -> 0
- net NRST: track 24.5 -> 0.00 mm
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
Commit message: Hmmm
Parts:
- moved J3 24.1 mm to (158.1, 97.8), turned to 90 degrees
- moved SW2 8.35 mm to (131.4, 99.7), turned to 0 degrees
- moved C10 4.66 mm to (136.5, 99.1)
- moved Y1 4.07 mm to (136.5, 102.2)
- moved C11 3.59 mm to (136.5, 105.4)
- moved SW1 1.27 mm to (131.4, 104.1), turned to 0 degrees
- moved C1 0.64 mm to (163.8, 103.5)
- moved C3 0.64 mm to (157.5, 103.5)
- moved U1 0.64 mm to (160.7, 103.5)
Routing:
- net PB2: track 0.00 -> 16.2 mm
- net PB1: track 0.00 -> 14.5 mm
- net PB0: track 0.00 -> 12.0 mm
- net Net-(C10-Pad1): track 0.00 -> 10.6 mm
- net PC5: track 0.00 -> 9.59 mm
- net Net-(C11-Pad1): track 0.00 -> 9.22 mm
- net +3V3: track 0.00 -> 2.19 mm, vias 4 -> 0
- net SWO: vias 1 -> 0
- net SWDIO: vias 1 -> 0
- net SWCLK: vias 1 -> 0
- net SD_DET: vias 1 -> 0
- net SD_D3: vias 1 -> 0
- net SD_D2: vias 1 -> 0
- net SD_D1: vias 1 -> 0
- net SD_CMD: vias 1 -> 0
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
Commit message: Hmmm
Parts:
- added H1: ~, MountingHole:MountingHole_2.2mm_M2, F.Cu at (120.0, 110.5)
- added H2: ~, MountingHole:MountingHole_2.2mm_M2, F.Cu at (177.2, 110.5)
- added H3: ~, MountingHole:MountingHole_2.2mm_M2, F.Cu at (177.2, 85.1)
- added H4: ~, MountingHole:MountingHole_2.2mm_M2, F.Cu at (120.0, 85.1)
- J1: footprint stm32dev:USB_C_Receptacle_HRO_TYPE-C-31-M-12 -> Connector_USB:USB_C_Receptacle_HRO_TYPE-C-31-M-12
- moved R5 10.8 mm to (126.4, 102.9)
- moved J1 5.08 mm to (175.9, 97.8)
- moved J2 5.08 mm to (121.3, 100.3)
- moved C6 3.86 mm to (154.3, 90.2), turned to 0 degrees
- moved C13 2.90 mm to (157.5, 92.1)
- moved D1 2.01 mm to (161.9, 92.1), turned to 90 degrees
- moved C2 1.27 mm to (126.4, 104.1)
- moved R1 1.27 mm to (126.4, 105.4)
Other:
- board size 52.1 x 30.5 mm -> 62.2 x 30.5 mm

Commit message: Hmmmm
Parts:
- moved SW1 16.6 mm to (120.8, 91.5)
- moved D3 16.5 mm to (177.2, 106.7), turned to 180 degrees
- moved R6 15.6 mm to (177.2, 104.8)
- moved R9 12.1 mm to (177.2, 90.8)
- moved SW2 11.6 mm to (120.8, 104.2), turned to 180 degrees
- moved D4 9.71 mm to (177.2, 88.9), turned to 180 degrees
- moved D2 5.08 mm to (172.7, 104.8)

Commit message: Hmmm
Parts:
- D3: value YEL -> GR
- R1, R5: value NM -> 10k
- moved C2 12.8 mm to (125.1, 91.4)
- moved R1 12.8 mm to (125.1, 92.7)
- moved C3 5.75 mm to (163.2, 104.1)
- moved J3 5.72 mm to (163.8, 97.8)
- moved D1 5.71 mm to (167.6, 92.1), turned to 180 degrees
- moved U1 5.44 mm to (166.1, 104.1)
- moved R2 5.20 mm to (169.0, 97.2)
- moved R8 5.20 mm to (169.0, 95.9)
- moved C1 5.12 mm to (168.9, 104.1)
- moved R3 5.08 mm to (168.9, 98.4)
- moved R7 5.08 mm to (168.9, 99.7)
- moved R5 2.29 mm to (125.1, 104.8)
Routing:
- net PB2: track 16.2 -> 0.00 mm
- net PB1: track 14.5 -> 0.00 mm
- net PB0: track 12.0 -> 0.00 mm
- net PC5: track 9.59 -> 0.00 mm

Commit message: Hmmm
Parts:
- moved C4 17.9 mm to (160.7, 96.5)
- moved SW1 14.0 mm to (128.9, 102.9), turned to 90 degrees
- moved R1 12.9 mm to (120.7, 104.8)
- moved C2 12.9 mm to (120.7, 103.5)
- moved R5 4.62 mm to (120.7, 106.0)
- moved SW2 4.56 mm to (125.1, 102.9), turned to 90 degrees
- moved C10 3.70 mm to (133.3, 101.0), turned to 180 degrees
- moved C11 3.70 mm to (133.3, 103.5)
- moved C9 2.54 mm to (146.1, 104.8), turned to 180 degrees
Routing:
- net PC0: track 0.00 -> 24.5 mm
- net PC1: track 0.00 -> 22.1 mm
- net PC2: track 0.00 -> 19.8 mm
- net PC3: track 0.00 -> 17.5 mm
- net PA0: track 0.00 -> 15.6 mm
- net PA1: track 0.00 -> 13.2 mm
- net PA4: track 0.00 -> 12.7 mm
- net PA5: track 0.00 -> 11.2 mm
- net PA3: track 0.00 -> 11.1 mm
- net PA2: track 0.00 -> 11.0 mm
- net PA6: track 0.00 -> 9.45 mm
- net PA7: track 0.00 -> 7.72 mm
- net Net-(C11-Pad1): track 9.22 -> 13.5 mm
- net PC4: track 0.00 -> 2.54 mm
- net +3V3: track 2.19 -> 4.30 mm
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