File: pcb/stm32dev.sch (KiCad schematic (older format))
At the start: 29 parts, among them J1 USB_B_Micro, J2 Micro_SD_Card_Det, U1 AMS1117-3.3, U2 STM32F405RGTx, Y1 16 MHz

Commit message: Hmmmmm
Parts:
- removed R1, R4: 10k, Resistor_SMD:R_0402_1005Metric, symbol Device:R
- removed U1: AMS1117-3.3, Package_TO_SOT_SMD:SOT-223-3_TabPin2, symbol Regulator_Linear:AMS1117-3.3
- removed Y1: 16 MHz, Crystal:Crystal_SMD_3225-4Pin_3.2x2.5mm, symbol Device:Crystal_GND24
- added C11: 1uF, Capacitor_SMD:C_0402_1005Metric, symbol Device:C
- added U1: XC6206P332MR, Package_TO_SOT_SMD:SOT-23, symbol Regulator_Linear:XC6206PxxxMR
- added Y1: 8 MHz, Crystal:Crystal_SMD_Abracon_ABM3-2Pin_5.0x3.2mm, symbol Device:Crystal
- C10, C6: value 22pF -> 20pF; LCSC C1555 -> C1554
Connections:
- net labels added: +3.3V, PA10, PA11, PA12, PA13, PA14, PA15, PA2, PA3, PA4, PA5, PA6, PA7, PA8, PA9, PB0, PB1, PB10, PB11, PB12, PB13, PB14, PB15, PB2, PB3, PB4, PB6, PB7, PB8, PB9
- net labels removed: DM, DP
- wire segments 193 -> 203
- no-connect marks 14 -> 8
Other:
- moved on the sheet: C2, C4, C5, C7, C8, J2

Commit message: Hmmmm
Parts:
- removed C9: 100nF, Capacitor_SMD:C_0402_1005Metric, symbol Device:C
- removed D1: ~, Diode_SMD:D_SOD-123, symbol Device:D_Schottky
- removed J1: USB_B_Micro, Connector_USB:USB_Micro-B_Molex-105017-0001, symbol Connector:USB_B_Micro
- added D1: YEL, LED_SMD:LED_0603_1608Metric, symbol Device:LED
- added D4: ~, Diode_SMD:D_SOD-123, symbol Device:D_Schottky
- added D5: BLUE, LED_SMD:LED_0603_1608Metric, symbol Device:LED
- added J1: USB_C_Receptacle_USB2.0, Connector_USB:USB_C_Receptacle_HRO_TYPE-C-31-M-12, symbol Connector:USB_C_Receptacle_USB2.0
- added R1: NM, Resistor_SMD:R_0402_1005Metric, symbol Device:R
- added R4: 22R, Resistor_SMD:R_0402_1005Metric, symbol Device:R
- added R5: 1.5k, Resistor_SMD:R_0402_1005Metric, symbol Device:R
- added R6, R8: 1k, Resistor_SMD:R_0402_1005Metric, symbol Device:R
- added R7, R9: 5.1k, Resistor_SMD:R_0402_1005Metric, symbol Device:R
- J5: footprint Connector_PinHeader_2.54mm:PinHeader_1x06_P2.54mm_Vertical -> Connector_PinHeader_2.54mm:PinHeader_1x06_P2.54mm_Horizontal
- R2: value 22R -> NM; LCSC C25092 -> (none)
Connections:
- net labels added: +5V, C13
- net labels removed: VCC
- wire segments 203 -> 232
- no-connect marks 8 -> 11
Other:
- note added: "Internal pull-up"
- note added: "USB C Connection"
- moved on the sheet: C10, C12, C13, C6, D3, J2, J5, U2

Commit message: Hmmmm
Connections:
- net labels added: PB5
Other:
- moved on the sheet: C3, D2, J2

Commit message: Hmmm
Connections:
- net labels added: PC0, PC1, PC13, PC14, PC15, PC2, PC3, PC4, PC5, SWCLK, SWDIO, SWO
- net labels removed: 0, EN, PA13, PA13_JMS, PA14, PA14_JCLK, PA15_JDI, PA2_U2_TX, PA3_U2_RX, PA4_AO0, PA5_AO1, PA6_AI0, PA7_AI1, PB10_SCK, PB12_CAN2_RX, PB13_CAN2_TX, PB3, PB3_JDO, PB4_JRST, PB6_SCL, PB7_SDA, PB8_CAN1_TX, PB9_CAN1_RX, PC2_MISO, PC3_MOSI, PC7, RGB, RXD, TXD
- wire segments 232 -> 248
- no-connect marks 11 -> 4
Other:
- moved on the sheet: D2

Commit message: Hmmm
Parts:
- removed D3: ~, Diode_SMD:D_SOD-123, symbol Device:D_Schottky
Connections:
- wire segments 248 -> 247
Other:
- moved on the sheet: C10, C11, C4, C5, C6, C7, C8
