File: pcb/stm32dev.sch (KiCad schematic (older format))
At the start: 36 parts, among them J1 USB_C_Receptacle_USB2.0, J3 Micro_SD_Card_Det, U1 XC6206P332MR, U2 STM32F405RGTx, Y1 8 MHz

Commit message: Hmmmm
Parts:
- J1: symbol Connector:USB_C_Receptacle_USB2.0 -> stm32dev-rescue:USB_C_Receptacle_USB2.0-Connector
Changed lines of the file:
@@
 $EndComp
 $Comp
-L Connector:USB_C_Receptacle_USB2.0 J1
+L stm32dev-rescue:USB_C_Receptacle_USB2.0-Connector J1
 U 1 1 5F19076D
 P 1100 6250

Commit message: Hmmmm
Parts:
- added AE1: Antenna_Shield, Connector_Coaxial:U.FL_Molex_MCRF_73412-0110_Vertical, symbol Device:Antenna_Shield
- added U3: NRF24L01, Package_DFN_QFN:QFN-20-1EP_4x4mm_P0.5mm_EP2.5x2.5mm, symbol RF:NRF24L01
- SW1, SW2: footprint Button_Switch_SMD:SW_SPST_TL3342 -> Button_Switch_SMD:SW_Push_1P1T_NO_CK_KMR2; LCSC C318887 -> C498310
Other:
- moved on the sheet: C10, C11, J3
Changed lines of the file:
@@
 L Device:C C10
 U 1 1 61FD3F87
-P 4650 3350
-F 0 "C10" H 4650 3450 50  0000 L CNN
-F 1 "20pF" H 4650 3250 50  0000 L CNN
-F 2 "Capacitor_SMD:C_0402_1005Metric" H 4688 3200 50  0001 C CNN
-F 3 "~" H 4650 3350 50  0001 C CNN
-F 4 "" H 4650 3350 50  0001 C CNN "LSCS"
-F 5 "C1554" H 4650 3350 50  0001 C CNN "LCSC"
-	1    4650 3350
+P 5150 3350
+F 0 "C10" H 5150 3450 50  0000 L CNN
+F 1 "20pF" H 5150 3250 50  0000 L CNN
+F 2 "Capacitor_SMD:C_0402_1005Metric" H 5188 3200 50  0001 C CNN
+F 3 "~" H 5150 3350 50  0001 C CNN
+F 4 "" H 5150 3350 50  0001 C CNN "LSCS"
+F 5 "C1554" H 5150 3350 50  0001 C CNN "LCSC"
+	1    5150 3350
 	1    0    0    -1
 $EndComp
@@
 L Device:C C11
 U 1 1 61FD4A27
-P 5450 3350
-F 0 "C11" H 5450 3450 50  0000 L CNN
-F 1 "20pF" H 5450 3250 50  0000 L CNN
-F 2 "Capacitor_SMD:C_0402_1005Metric" H 5488 3200 50  0001 C CNN
-F 3 "~" H 5450 3350 50  0001 C CNN
-F 4 "" H 5450 3350 50  0001 C CNN "LSCS"
-F 5 "C1554" H 5450 3350 50  0001 C CNN "LCSC"
-	1    5450 3350
+P 5950 3350
+F 0 "C11" H 5950 3450 50  0000 L CNN
+F 1 "20pF" H 5950 3250 50  0000 L CNN
+F 2 "Capacitor_SMD:C_0402_1005Metric" H 5988 3200 50  0001 C CNN
+F 3 "~" H 5950 3350 50  0001 C CNN
+F 4 "" H 5950 3350 50  0001 C CNN "LSCS"
+F 5 "C1554" H 5950 3350 50  0001 C CNN "LCSC"
+	1    5950 3350
 	1    0    0    -1
 $EndComp
@@
 L power:GND #PWR023
 U 1 1 61FD9C31
-P 4650 3600
-F 0 "#PWR023" H 4650 3350 50  0001 C CNN
-F 1 "GND" H 4655 3427 50  0000 C CNN
-F 2 "" H 4650 3600 50  0001 C CNN
-F 3 "" H 4650 3600 50  0001 C CNN
-	1    4650 3600
+P 5150 3600
+F 0 "#PWR023" H 5150 3350 50  0001 C CNN
+F 1 "GND" H 5155 3427 50  0000 C CNN
+F 2 "" H 5150 3600 50  0001 C CNN
+F 3 "" H 5150 3600 50  0001 C CNN
+	1    5150 3600
 	1    0    0    -1
 $EndComp
@@
 L power:GND #PWR026
 U 1 1 61FDD0AD
-P 5450 3600
-F 0 "#PWR026" H 5450 3350 50  0001 C CNN
-F 1 "GND" H 5455 3427 50  0000 C CNN
-F 2 "" H 5450 3600 50  0001 C CNN
-F 3 "" H 5450 3600 50  0001 C CNN
-	1    5450 3600
-	1    0    0    -1
-$EndComp
-Wire Wire Line
-	4650 3500 4650 3600
-Wire Wire Line
-	5450 3500 5450 3600
-Wire Wire Line
-	5200 3000 5450 3000
-Wire Wire Line
-	5450 3000 5450 3200
-Wire Wire Line
-	4900 3000 4650 3000
-Wire Wire Line
-	4650 3000 4650 3200
-Wire Wire Line
-	6750 2700 5450 2700
-Wire Wire Line
-	5450 2700 5450 3000
-Connection ~ 5450 3000
-Wire Wire Line
-	6750 2600 4650 2600
-Wire Wire Line
-	4650 2600 4650 3000
-Connection ~ 4650 3000
+P 5950 3600
+F 0 "#PWR026" H 5950 3350 50  0001 C CNN
+F 1 "GND" H 5955 3427 50  0000 C CNN
+F 2 "" H 5950 3600 50  0001 C CNN
+F 3 "" H 5950 3600 50  0001 C CNN
+	1    5950 3600
+	1    0    0    -1
+$EndComp
+Wire Wire Line
+	5150 3500 5150 3600
+Wire Wire Line
+	5950 3500 5950 3600
+Wire Wire Line
+	5700 3000 5950 3000
+Wire Wire Line
+	5950 3000 5950 3200
+Wire Wire Line
+	5400 3000 5150 3000
+Wire Wire Line
+	5150 3000 5150 3200
+Wire Wire Line
+	6750 2700 5950 2700
+Wire Wire Line
+	5950 2700 5950 3000
+Connection ~ 5950 3000
+Wire Wire Line
+	6750 2600 5150 2600
+Wire Wire Line
+	5150 2600 5150 3000
+Connection ~ 5150 3000
 $Comp
 L Device:C C5
@@
 L Connector:Micro_SD_Card_Det J3
 U 1 1 62026105
-P 5700 6350
-F 0 "J3" H 5650 7167 50  0000 C CNN
-F 1 "Micro_SD_Card_Det" H 5650 7076 50  0000 C CNN
-F 2 "Connector_Card:microSD_HC_Hirose_DM3D-SF" H 7750 7050 50  0001 C CNN
-F 3 "https://www.hirose.com/product/en/download_file/key_name/DM3/category/Catalog/doc_file_id/49662/?file_category_id=4&item_id=195&is_series=1" H 5700 6450 50  0001 C CNN
-	1    5700 6350
+P 5650 6850
+F 0 "J3" H 5600 7667 50  0000 C CNN
+F 1 "Micro_SD_Card_Det" H 5600 7576 50  0000 C CNN
+F 2 "Connector_Card:microSD_HC_Hirose_DM3D-SF" H 7700 7550 50  0001 C CNN
+F 3 "https://www.hirose.com/product/en/download_file/key_name/DM3/category/Catalog/doc_file_id/49662/?file_category_id=4&item_id=195&is_series=1" H 5650 6950 50  0001 C CNN
+	1    5650 6850
 	1    0    0    -1
 $EndComp
@@
 	1    0    0    -1
 $EndComp
-Text GLabel 4600 5950 0    50   Input ~ 0
+Text GLabel 4550 6450 0    50   Input ~ 0
 SD_D2
-Text GLabel 4600 6050 0    50   Input ~ 0
+Text GLabel 4550 6550 0    50   Input ~ 0
 SD_D3
-Text GLabel 4600 6150 0    50   Input ~ 0
+Text GLabel 4550 6650 0    50   Input ~ 0
 SD_CMD
-Text GLabel 4600 6350 0    50   Input ~ 0
+Text GLabel 4550 6850 0    50   Input ~ 0
 SD_CLK
-Text GLabel 4600 6550 0    50   Input ~ 0
+Text GLabel 4550 7050 0    50   Input ~ 0
 SD_D0
-Text GLabel 4600 6650 0    50   Input ~ 0
+Text GLabel 4550 7150 0    50   Input ~ 0
 SD_D1
-Text GLabel 4600 6750 0    50   Input ~ 0
+Text GLabel 4550 7250 0    50   Input ~ 0
 SD_DET
 Wire Wire Line
-	4600 5950 4800 5950
-Wire Wire Line
-	4800 6050 4600 6050
-Wire Wire Line
-	4600 6150 4800 6150
-Wire Wire Line
-	4800 6350 4600 6350
-Wire Wire Line
-	4600 6550 4800 6550
-Wire Wire Line
-	4600 6650 4800 6650
-Wire Wire Line
-	4800 6750 4600 6750
+	4550 6450 4750 6450
+Wire Wire Line
+	4750 6550 4550 6550
+Wire Wire Line
+	4550 6650 4750 6650
+Wire Wire Line
+	4750 6850 4550 6850
+Wire Wire Line
+	4550 7050 4750 7050
+Wire Wire Line
+	4550 7150 4750 7150
+Wire Wire Line
+	4750 7250 4550 7250
 $Comp
 L power:GND #PWR025
 U 1 1 62151480
-P 4700 6950
-F 0 "#PWR025" H 4700 6700 50  0001 C CNN
-F 1 "GND" H 4705 6777 50  0000 C CNN
-F 2 "" H 4700 6950 50  0001 C CNN
-F 3 "" H 4700 6950 50  0001 C CNN
-	1    4700 6950
-	1    0    0    -1
-$EndComp
-Wire Wire Line
-	4700 5800 4700 6250
-Wire Wire Line
-	4700 6250 4800 6250
-Wire Wire Line
-	4800 6450 4700 6450
-Wire Wire Line
-	4700 6450 4700 6850
-Wire Wire Line
-	4800 6850 4700 6850
-Connection ~ 4700 6850
-Wire Wire Line
-	4700 6850 4700 6950
+P 4650 7450
+F 0 "#PWR025" H 4650 7200 50  0001 C CNN
+F 1 "GND" H 4655 7277 50  0000 C CNN
+F 2 "" H 4650 7450 50  0001 C CNN
+F 3 "" H 4650 7450 50  0001 C CNN
+	1    4650 7450
+	1    0    0    -1
+$EndComp
+Wire Wire Line
+	4650 6300 4650 6750
+Wire Wire Line
+	4650 6750 4750 6750
+Wire Wire Line
+	4750 6950 4650 6950
+Wire Wire Line
+	4650 6950 4650 7350
+Wire Wire Line
+	4750 7350 4650 7350
+Connection ~ 4650 7350
+Wire Wire Line
+	4650 7350 4650 7450
 Text GLabel 6650 4100 0    50   Input ~ 0
 SD_D2
@@
 L power:GND #PWR029
 U 1 1 623690A3
-P 6600 6950
-F 0 "#PWR029" H 6600 6700 50  0001 C CNN
-F 1 "GND" H 6605 6777 50  0000 C CNN
-F 2 "" H 6600 6950 50  0001 C CNN
-F 3 "" H 6600 6950 50  0001 C CNN
-	1    6600 6950
-	1    0    0    -1
-$EndComp
-Wire Wire Line
-	6500 6850 6600 6850
-Wire Wire Line
-	6600 6850 6600 6950
+P 6550 7450
+F 0 "#PWR029" H 6550 7200 50  0001 C CNN
+F 1 "GND" H 6555 7277 50  0000 C CNN
+F 2 "" H 6550 7450 50  0001 C CNN
+F 3 "" H 6550 7450 50  0001 C CNN
+	1    6550 7450
+	1    0    0    -1
+$EndComp
+Wire Wire Line
+	6450 7350 6550 7350
+Wire Wire Line
+	6550 7350 6550 7450
 Text GLabel 6650 3800 0    50   Input ~ 0
 SD_DET
@@
 L Device:Crystal Y1
 U 1 1 5F0B081F
-P 5050 3000
-F 0 "Y1" H 5050 3268 50  0000 C CNN
-F 1 "8 MHz" H 5050 3177 50  0000 C CNN
-F 2 "Crystal:Crystal_SMD_Abracon_ABM3-2Pin_5.0x3.2mm" H 5050 3000 50  0001 C CNN
-F 3 "~" H 5050 3000 50  0001 C CNN
-F 4 "C115962" H 5050 3000 50  0001 C CNN "LCSC"
-	1    5050 3000
+P 5550 3000
+F 0 "Y1" H 5550 3268 50  0000 C CNN
+F 1 "8 MHz" H 5550 3177 50  0000 C CNN
+F 2 "Crystal:Crystal_SMD_Abracon_ABM3-2Pin_5.0x3.2mm" H 5550 3000 50  0001 C CNN
+F 3 "~" H 5550 3000 50  0001 C CNN
+F 4 "C115962" H 5550 3000 50  0001 C CNN "LCSC"
+	1    5550 3000
 	1    0    0    -1
 $EndComp
@@
 L power:+3.3V #PWR024
 U 1 1 5F0BE1E9
-P 4700 5800
-F 0 "#PWR024" H 4700 5650 50  0001 C CNN
-F 1 "+3.3V" H 4715 5973 50  0000 C CNN
-F 2 "" H 4700 5800 50  0001 C CNN
-F 3 "" H 4700 5800 50  0001 C CNN
-	1    4700 5800
+P 4650 6300
+F 0 "#PWR024" H 4650 6150 50  0001 C CNN
+F 1 "+3.3V" H 4665 6473 50  0000 C CNN
+F 2 "" H 4650 6300 50  0001 C CNN
+F 3 "" H 4650 6300 50  0001 C CNN
+	1    4650 6300
 	1    0    0    -1
 $EndComp
@@
 F 0 "SW1" H 1100 3000 50  0000 C CNN
 F 1 "~" H 1400 3000 50  0000 C CNN
-F 2 "Button_Switch_SMD:SW_SPST_TL3342" H 1200 3100 50  0001 C CNN
+F 2 "Button_Switch_SMD:SW_Push_1P1T_NO_CK_KMR2" H 1200 3100 50  0001 C CNN
 F 3 "https://datasheet.lcsc.com/szlcsc/1901111503_XKB-Enterprise-TS-1187A-B-A-B_C318884.pdf" H 1200 3100 50  0001 C CNN
-F 4 "C318887" H 1200 2900 50  0001 C CNN "LCSC"
+F 4 "C498310" H 1200 2900 50  0001 C CNN "LCSC"
 	1    1200 2900
 	0    -1   -1   0
@@
 F 0 "SW2" H 2150 2550 50  0000 C CNN
 F 1 "~" H 2450 2550 50  0000 C CNN
-F 2 "Button_Switch_SMD:SW_SPST_TL3342" H 2250 2650 50  0001 C CNN
+F 2 "Button_Switch_SMD:SW_Push_1P1T_NO_CK_KMR2" H 2250 2650 50  0001 C CNN
 F 3 "https://datasheet.lcsc.com/szlcsc/1901111503_XKB-Enterprise-TS-1187A-B-A-B_C318884.pdf" H 2250 2650 50  0001 C CNN
-F 4 "C318887" H 2250 2450 50  0001 C CNN "LCSC"
+F 4 "C498310" H 2250 2450 50  0001 C CNN "LCSC"
 	1    2250 2450
 	0    -1   -1   0
@@
 	1    0    0    -1
 $EndComp
+$Comp
+L Device:Antenna_Shield AE1
+U 1 1 5FDECA55
+P 13250 2900
+F 0 "AE1" H 13394 2939 50  0000 L CNN
+F 1 "Antenna_Shield" H 13394 2848 50  0000 L CNN
+F 2 "Connector_Coaxial:U.FL_Molex_MCRF_73412-0110_Vertical" H 13250 3000 50  0001 C CNN
+F 3 "~" H 13250 3000 50  0001 C CNN
+	1    13250 2900
+	1    0    0    -1
+$EndComp
+$Comp
+L RF:NRF24L01 U3
+U 1 1 5FDEEEC0
+P 14450 4500
+F 0 "U3" H 14450 5481 50  0000 C CNN
+F 1 "NRF24L01" H 14450 5390 50  0000 C CNN
+F 2 "Package_DFN_QFN:QFN-20-1EP_4x4mm_P0.5mm_EP2.5x2.5mm" H 14650 5300 50  0001 L CIN
+F 3 "http://www.nordicsemi.com/eng/content/download/2730/34105/file/nRF24L01_Product_Specification_v2_0.pdf" H 14450 4600 50  0001 C CNN
+	1    14450 4500
+	1    0    0    -1
+$EndComp

Commit message: Hmmm
Parts:
- added C14, C15: 20pF, Capacitor_SMD:C_0402_1005Metric, symbol Device:C
- added C16: 1.5pF, Capacitor_SMD:C_0402_1005Metric, symbol Device:C
- added C17: 1pF, Capacitor_SMD:C_0402_1005Metric, symbol Device:C
- added L1: 8.2nH, Inductor_SMD:L_0402_1005Metric, symbol Device:L
- added L2: 2.7nH, Inductor_SMD:L_0402_1005Metric, symbol Device:L
- added L3: 3.9nH, Inductor_SMD:L_0402_1005Metric, symbol Device:L
- added R10: 1M, Resistor_SMD:R_0402_1005Metric, symbol Device:R
- added Y2: 16MHz, Crystal:Crystal_SMD_3225-4Pin_3.2x2.5mm, symbol Device:Crystal_GND24
- AE1: footprint Connector_Coaxial:U.FL_Molex_MCRF_73412-0110_Vertical -> Connector_Coaxial:U.FL_Hirose_U.FL-R-SMT-1_Vertical; LCSC (none) -> C88374
- U3: LCSC (none) -> C8791
Connections:
- wire segments 285 -> 340

Commit message: Hmmm
Parts:
- removed R4: 1.5k, Resistor_SMD:R_0402_1005Metric, symbol Device:R
- removed Y1: 8 MHz, Crystal:Crystal_SMD_Abracon_ABM3-2Pin_5.0x3.2mm, symbol Device:Crystal
- added Y1: 16MHz, Crystal:Crystal_SMD_3225-4Pin_3.2x2.5mm, symbol Device:Crystal_GND24
Connections:
- wire segments 340 -> 341
Other:
- moved on the sheet: C10, C11
Changed lines of the file:
@@
 L Device:C C10
 U 1 1 61FD3F87
-P 5150 3350
-F 0 "C10" H 5150 3450 50  0000 L CNN
-F 1 "20pF" H 5150 3250 50  0000 L CNN
-F 2 "Capacitor_SMD:C_0402_1005Metric" H 5188 3200 50  0001 C CNN
-F 3 "~" H 5150 3350 50  0001 C CNN
-F 4 "" H 5150 3350 50  0001 C CNN "LSCS"
-F 5 "C1554" H 5150 3350 50  0001 C CNN "LCSC"
-	1    5150 3350
+P 4950 3600
+F 0 "C10" H 4950 3700 50  0000 L CNN
+F 1 "20pF" H 4950 3500 50  0000 L CNN
+F 2 "Capacitor_SMD:C_0402_1005Metric" H 4988 3450 50  0001 C CNN
+F 3 "~" H 4950 3600 50  0001 C CNN
+F 4 "" H 4950 3600 50  0001 C CNN "LSCS"
+F 5 "C1554" H 4950 3600 50  0001 C CNN "LCSC"
+	1    4950 3600
 	1    0    0    -1
 $EndComp
@@
 L Device:C C11
 U 1 1 61FD4A27
-P 5950 3350
-F 0 "C11" H 5950 3450 50  0000 L CNN
-F 1 "20pF" H 5950 3250 50  0000 L CNN
-F 2 "Capacitor_SMD:C_0402_1005Metric" H 5988 3200 50  0001 C CNN
-F 3 "~" H 5950 3350 50  0001 C CNN
-F 4 "" H 5950 3350 50  0001 C CNN "LSCS"
-F 5 "C1554" H 5950 3350 50  0001 C CNN "LCSC"
-	1    5950 3350
+P 5600 3600
+F 0 "C11" H 5600 3700 50  0000 L CNN
+F 1 "20pF" H 5600 3500 50  0000 L CNN
+F 2 "Capacitor_SMD:C_0402_1005Metric" H 5638 3450 50  0001 C CNN
+F 3 "~" H 5600 3600 50  0001 C CNN
+F 4 "" H 5600 3600 50  0001 C CNN "LSCS"
+F 5 "C1554" H 5600 3600 50  0001 C CNN "LCSC"
+	1    5600 3600
 	1    0    0    -1
 $EndComp
@@
 L power:GND #PWR023
 U 1 1 61FD9C31
-P 5150 3600
-F 0 "#PWR023" H 5150 3350 50  0001 C CNN
-F 1 "GND" H 5155 3427 50  0000 C CNN
-F 2 "" H 5150 3600 50  0001 C CNN
-F 3 "" H 5150 3600 50  0001 C CNN
-	1    5150 3600
+P 4950 3850
+F 0 "#PWR023" H 4950 3600 50  0001 C CNN
+F 1 "GND" H 4955 3677 50  0000 C CNN
+F 2 "" H 4950 3850 50  0001 C CNN
+F 3 "" H 4950 3850 50  0001 C CNN
+	1    4950 3850
 	1    0    0    -1
 $EndComp
@@
 L power:GND #PWR026
 U 1 1 61FDD0AD
-P 5950 3600
-F 0 "#PWR026" H 5950 3350 50  0001 C CNN
-F 1 "GND" H 5955 3427 50  0000 C CNN
-F 2 "" H 5950 3600 50  0001 C CNN
-F 3 "" H 5950 3600 50  0001 C CNN
-	1    5950 3600
-	1    0    0    -1
-$EndComp
-Wire Wire Line
-	5150 3500 5150 3600
-Wire Wire Line
-	5950 3500 5950 3600
-Wire Wire Line
-	5700 3000 5950 3000
-Wire Wire Line
-	5950 3000 5950 3200
-Wire Wire Line
-	5400 3000 5150 3000
-Wire Wire Line
-	5150 3000 5150 3200
-Wire Wire Line
-	6750 2700 5950 2700
-Wire Wire Line
-	5950 2700 5950 3000
-Connection ~ 5950 3000
-Wire Wire Line
-	6750 2600 5150 2600
-Wire Wire Line
-	5150 2600 5150 3000
-Connection ~ 5150 3000
+P 5600 3850
+F 0 "#PWR026" H 5600 3600 50  0001 C CNN
+F 1 "GND" H 5605 3677 50  0000 C CNN
+F 2 "" H 5600 3850 50  0001 C CNN
+F 3 "" H 5600 3850 50  0001 C CNN
+	1    5600 3850
+	1    0    0    -1
+$EndComp
+Wire Wire Line
+	4950 3750 4950 3850
+Wire Wire Line
+	5600 3750 5600 3850
+Wire Wire Line
+	5400 3300 5600 3300
+Wire Wire Line
+	5600 3300 5600 3450
+Wire Wire Line
+	5100 3300 4950 3300
+Wire Wire Line
+	4950 3300 4950 3450
+Wire Wire Line
+	6750 2700 5600 2700
+Wire Wire Line
+	5600 2700 5600 3300
+Connection ~ 5600 3300
+Wire Wire Line
+	6750 2600 4950 2600
+Wire Wire Line
+	4950 2600 4950 3300
+Connection ~ 4950 3300
 $Comp
 L Device:C C5
@@
 L power:GND #PWR013
 U 1 1 6204BB30
-P 2900 4450
-F 0 "#PWR013" H 2900 4200 50  0001 C CNN
-F 1 "GND" H 2905 4277 50  0000 C CNN
-F 2 "" H 2900 4450 50  0001 C CNN
-F 3 "" H 2900 4450 50  0001 C CNN
-	1    2900 4450
-	1    0    0    -1
-$EndComp
-Wire Wire Line
-	3000 4250 2900 4250
-Wire Wire Line
-	3500 4250 3600 4250
-Wire Wire Line
-	3000 4350 2900 4350
-Wire Wire Line
-	2900 4350 2900 4450
-Wire Wire Line
-	3600 4350 3500 4350
+P 9750 6250
+F 0 "#PWR013" H 9750 6000 50  0001 C CNN
+F 1 "GND" H 9755 6077 50  0000 C CNN
+F 2 "" H 9750 6250 50  0001 C CNN
+F 3 "" H 9750 6250 50  0001 C CNN
+	1    9750 6250
+	1    0    0    -1
+$EndComp
+Wire Wire Line
+	9850 6050 9750 6050
+Wire Wire Line
+	10350 6050 10450 6050
+Wire Wire Line
+	9850 6150 9750 6150
+Wire Wire Line
+	9750 6150 9750 6250
+Wire Wire Line
+	10450 6150 10350 6150
 $Comp
 L LED:WS2812B D1
@@
 	10200 5200 10300 5200
 Wire Wire Line
-	3500 4150 3600 4150
+	10350 5950 10450 5950
 Wire Wire Line
 	2950 950  3250 950
@@
 Wire Wire Line
 	8250 2500 8150 2500
-$Comp
-L Device:Crystal Y1
-U 1 1 5F0B081F
-P 5550 3000
-F 0 "Y1" H 5550 3268 50  0000 C CNN
-F 1 "8 MHz" H 5550 3177 50  0000 C CNN
-F 2 "Crystal:Crystal_SMD_Abracon_ABM3-2Pin_5.0x3.2mm" H 5550 3000 50  0001 C CNN
-F 3 "~" H 5550 3000 50  0001 C CNN
-F 4 "C115962" H 5550 3000 50  0001 C CNN "LCSC"
-	1    5550 3000
-	1    0    0    -1
-$EndComp
 $Comp
 L Regulator_Linear:XC6206PxxxMR U1
@@
 Wire Wire Line
 	1800 6150 2000 6150
-$Comp
-L Device:R R4
-U 1 1 5F1907BD
-P 2150 6450
-F 0 "R4" V 2200 6600 50  0000 L CNN
-F 1 "1.5k" V 2200 6150 50  0000 L CNN
-F 2 "Resistor_SMD:R_0402_1005Metric" V 2080 6450 50  0001 C CNN
-F 3 "~" H 2150 6450 50  0001 C CNN
-F 4 "C25867" H 2150 6450 50  0001 C CNN "LCSC"
-	1    2150 6450
-	0    -1   -1   0
-$EndComp
-Wire Wire Line
-	2000 6450 1800 6450
-Connection ~ 1800 6450
-$Comp
-L power:+3.3V #PWR011
-U 1 1 5F1907C5
-P 2550 5550
-F 0 "#PWR011" H 2550 5400 50  0001 C CNN
-F 1 "+3.3V" H 2565 5723 50  0000 C CNN
-F 2 "" H 2550 5550 50  0001 C CNN
-F 3 "" H 2550 5550 50  0001 C CNN
-	1    2550 5550
-	1    0    0    -1
-$EndComp
-Wire Wire Line
-	2550 5550 2550 6450
-Wire Wire Line
-	2550 6450 2300 6450
 Wire Notes Line
 	650  7650 4000 7650
@@
 Text GLabel 8250 3600 2    50   Input ~ 0
 PB5
-Text GLabel 2900 4250 0    50   Input ~ 0
+Text GLabel 9750 6050 0    50   Input ~ 0
 SWCLK
-Text GLabel 3600 4250 2    50   Input ~ 0
+Text GLabel 10450 6050 2    50   Input ~ 0
 SWDIO
-Text GLabel 3600 4350 2    50   Input ~ 0
+Text GLabel 10450 6150 2    50   Input ~ 0
 SWO
 Text GLabel 6650 3100 0    50   Input ~ 0
@@
 L power:+3.3V #PWR021
 U 1 1 5F78FF2D
-P 3600 4050
-F 0 "#PWR021" H 3600 3900 50  0001 C CNN
-F 1 "+3.3V" H 3615 4223 50  0000 C CNN
-F 2 "" H 3600 4050 50  0001 C CNN
-F 3 "" H 3600 4050 50  0001 C CNN
-	1    3600 4050
-	1    0    0    -1
-$EndComp
-Wire Wire Line
-	3600 4050 3600 4150
-Text GLabel 2900 4150 0    50   Input ~ 0
+P 10450 5850
+F 0 "#PWR021" H 10450 5700 50  0001 C CNN
+F 1 "+3.3V" H 10465 6023 50  0000 C CNN
+F 2 "" H 10450 5850 50  0001 C CNN
+F 3 "" H 10450 5850 50  0001 C CNN
+	1    10450 5850
+	1    0    0    -1
+$EndComp
+Wire Wire Line
+	10450 5850 10450 5950
+Text GLabel 9750 5950 0    50   Input ~ 0
 NRST
 Wire Wire Line
-	2900 4150 3000 4150
+	9750 5950 9850 5950
 $Comp
 L power:+5V #PWR032
@@
 L Connector_Generic:Conn_02x03_Odd_Even J2
 U 1 1 5F3A1665
-P 3200 4250
-F 0 "J2" H 3250 4475 50  0000 C CNN
-F 1 "~" H 3250 4476 50  0000 C CNN
-F 2 "Connector_PinHeader_2.54mm:PinHeader_2x03_P2.54mm_Horizontal" H 3200 4250 50  0001 C CNN
-F 3 "~" H 3200 4250 50  0001 C CNN
-	1    3200 4250
+P 10050 6050
+F 0 "J2" H 10100 6275 50  0000 C CNN
+F 1 "~" H 10100 6276 50  0000 C CNN
+F 2 "Connector_PinHeader_2.54mm:PinHeader_2x03_P2.54mm_Horizontal" H 10050 6050 50  0001 C CNN
+F 3 "~" H 10050 6050 50  0001 C CNN
+	1    10050 6050
 	1    0    0    -1
 $EndComp
@@
 Wire Wire Line
 	15800 4200 15700 4200
+$Comp
+L Device:Crystal_GND24 Y1
+U 1 1 6010DF9D
+P 5250 3300
+F 0 "Y1" H 5450 3200 50  0000 R CNN
+F 1 "16MHz" H 5150 3200 50  0000 R CNN
+F 2 "Crystal:Crystal_SMD_3225-4Pin_3.2x2.5mm" H 5250 3300 50  0001 C CNN
+F 3 "~" H 5250 3300 50  0001 C CNN
+F 4 "C13738" H 5250 3300 50  0001 C CNN "LCSC"
+	1    5250 3300
+	-1   0    0    1
+$EndComp
+$Comp
+L power:GND #PWR0105
+U 1 1 601981E2
+P 5250 3850
+F 0 "#PWR0105" H 5250 3600 50  0001 C CNN
+F 1 "GND" H 5255 3677 50  0000 C CNN
+F 2 "" H 5250 3850 50  0001 C CNN
+F 3 "" H 5250 3850 50  0001 C CNN
+	1    5250 3850
+	1    0    0    -1
+$EndComp
+Wire Wire Line
+	5250 3500 5250 3850
+$Comp
+L power:GND #PWR0106
+U 1 1 601B7626
+P 5900 3850
+F 0 "#PWR0106" H 5900 3600 50  0001 C CNN
+F 1 "GND" H 5905 3677 50  0000 C CNN
+F 2 "" H 5900 3850 50  0001 C CNN
+F 3 "" H 5900 3850 50  0001 C CNN
+	1    5900 3850
+	1    0    0    -1
+$EndComp
+Wire Wire Line
+	5900 3850 5900 3000
+Wire Wire Line
+	5900 3000 5250 3000
+Wire Wire Line
+	5250 3000 5250 3100
 $EndSCHEMATC

Commit message: Hmmm
Parts:
- removed R5: NM, Resistor_SMD:R_0402_1005Metric, symbol Device:R
- added JP1: ~, Jumper:SolderJumper-3_P1.3mm_Bridged2Bar12_Pad1.0x1.5mm, symbol Jumper:Jumper_3_Bridged12
- AE1: value Antenna_Shield -> ~
- R1: value NM -> 10k; LCSC (none) -> C25741
Connections:
- wire segments 341 -> 349
Other:
- note removed: "Internal pull-up"
- moved on the sheet: C10, C11, C12, C13, C14, C15, C16, C17, C2, C4, D1, D2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

Commit message: Removed all the wireless stuff - back to rev b
Parts:
- removed AE1: ~, Connector_Coaxial:U.FL_Hirose_U.FL-R-SMT-1_Vertical, symbol Device:Antenna_Shield
- removed C14, C15: 20pF, Capacitor_SMD:C_0402_1005Metric, symbol Device:C
- removed C16: 1.5pF, Capacitor_SMD:C_0402_1005Metric, symbol Device:C
- removed C17: 1pF, Capacitor_SMD:C_0402_1005Metric, symbol Device:C
- removed JP1: ~, Jumper:SolderJumper-3_P1.3mm_Bridged2Bar12_Pad1.0x1.5mm, symbol Jumper:Jumper_3_Bridged12
- removed L1: 8.2nH, Inductor_SMD:L_0402_1005Metric, symbol Device:L
- removed L2: 2.7nH, Inductor_SMD:L_0402_1005Metric, symbol Device:L
- removed L3: 3.9nH, Inductor_SMD:L_0402_1005Metric, symbol Device:L
- removed R10: 1M, Resistor_SMD:R_0402_1005Metric, symbol Device:R
- removed U3: NRF24L01, Package_DFN_QFN:QFN-20-1EP_4x4mm_P0.5mm_EP2.5x2.5mm, symbol RF:NRF24L01
- removed Y1, Y2: 16MHz, Crystal:Crystal_SMD_3225-4Pin_3.2x2.5mm, symbol Device:Crystal_GND24
- added R4: 1.5k, Resistor_SMD:R_0402_1005Metric, symbol Device:R
- added R5: NM, Resistor_SMD:R_0402_1005Metric, symbol Device:R
- added Y1: 8 MHz, Crystal:Crystal_SMD_Abracon_ABM3-2Pin_5.0x3.2mm, symbol Device:Crystal
- J1: symbol stm32dev-rescue:USB_C_Receptacle_USB2.0-Connector -> Connector:USB_C_Receptacle_USB2.0
- R1: value 10k -> NM; LCSC C25741 -> (none)
- SW1, SW2: footprint Button_Switch_SMD:SW_Push_1P1T_NO_CK_KMR2 -> Button_Switch_SMD:SW_SPST_TL3342; LCSC C498310 -> C318887
Connections:
- wire segments 349 -> 285
Other:
- note added: "Internal pull-up"
- moved on the sheet: C10, C11, C12, C13, C2, C4, D1, D2, J1, J3, U2
