File: pcb/stm32dev.sch (KiCad schematic (older format))
At the start: 35 parts, among them J3 Micro_SD_Card_Det, U1 XC6206P332MR, U2 STM32F405RGTx, Y1 16 MHz

Commit message: Hmmm
Parts:
- J1: footprint Connector_USB:USB_C_Receptacle_HRO_TYPE-C-31-M-12 -> stm32dev:USB_C_Receptacle_HRO_TYPE-C-31-M-12; symbol Connector:USB_C_Receptacle_USB2.0 -> stm32dev:USB_C_Receptacle_USB2.0; LCSC C167321 -> C165948
- SW2: footprint Button_Switch_SMD:SW_SPST_TL3342 -> stm32dev:TS-1088R-02526; symbol Switch:SW_Push -> stm32dev:TS-1088R-02526; LCSC C318887 -> C455281
Changed lines of the file:
@@
 $EndComp
 $Comp
-L Connector:USB_C_Receptacle_USB2.0 J1
+L stm32dev:USB_C_Receptacle_USB2.0 J1
 U 1 1 5F19076D
 P 1100 6250
 F 0 "J1" H 1207 7117 50  0000 C CNN
 F 1 "~" H 1207 7026 50  0001 C CNN
-F 2 "Connector_USB:USB_C_Receptacle_HRO_TYPE-C-31-M-12" H 1250 6250 50  0001 C CNN
-F 3 "https://datasheet.lcsc.com/szlcsc/1811101520_Jing-Extension-of-the-Electronic-Co-C167321_C167321.pdf" H 1250 6250 50  0001 C CNN
-F 4 "C167321" H 1100 6250 50  0001 C CNN "LCSC"
+F 2 "stm32dev:USB_C_Receptacle_HRO_TYPE-C-31-M-12" H 1250 6250 50  0001 C CNN
+F 3 "1811131825_Korean-Hroparts-Elec-TYPE-C-31-M-12_C165948.pdf" H 1250 6250 50  0001 C CNN
+F 4 "C165948" H 1100 6250 50  0001 C CNN "LCSC"
 	1    1100 6250
 	1    0    0    -1
@@
 $EndComp
 $Comp
-L Switch:SW_Push SW?
+L stm32dev:TS-1088R-02526 SW?
 U 1 1 5F1C1C5D
 P 2250 2450
@@
 F 0 "SW2" H 2150 2550 50  0000 C CNN
 F 1 "~" H 2450 2550 50  0000 C CNN
-F 2 "Button_Switch_SMD:SW_SPST_TL3342" H 2250 2650 50  0001 C CNN
-F 3 "https://datasheet.lcsc.com/szlcsc/1901111503_XKB-Enterprise-TS-1187A-B-A-B_C318884.pdf" H 2250 2650 50  0001 C CNN
-F 4 "C318887" H 2250 2450 50  0001 C CNN "LCSC"
+F 2 "stm32dev:TS-1088R-02526" H 2250 2650 50  0001 C CNN
+F 3 "https://datasheet.lcsc.com/szlcsc/1912111437_XUNPU-TS-1088R-02526_C455281.pdf" H 2250 2650 50  0001 C CNN
+F 4 "C455281" H 2250 2450 50  0001 C CNN "LCSC"
 	1    2250 2450
 	0    -1   -1   0

Commit message: Hmmm
Parts:
- added D?: ~, Diode_SMD:D_SOD-123, symbol Device:D_Schottky
- added D?: PSM712, Package_TO_SOT_SMD:SOT-23, symbol Power_Protection:SP0502BAHT
- added J?: USB_C_Receptacle_USB2.0, lifeline:USB_C_Receptacle_HRO_TYPE-C-31-M-12, symbol lifeline:USB_C_Receptacle_USB2.0
- added TP? (x2): ~, TestPoint:TestPoint_Pad_1.5x1.5mm, symbol Connector:TestPoint
- J1: footprint stm32dev:USB_C_Receptacle_HRO_TYPE-C-31-M-12 -> Connector_USB:USB_C_Receptacle_HRO_TYPE-C-31-M-12; symbol stm32dev:USB_C_Receptacle_USB2.0 -> Connector:USB_C_Receptacle_USB2.0; LCSC C165948 -> C167321
- SW2: symbol stm32dev:TS-1088R-02526 -> Switch:SW_Push
Connections:
- net labels added: CC1, CC2, HUDM, HUDP, VDC
- wire segments 287 -> 317
Changed lines of the file:
@@
 $EndComp
 $Comp
-L stm32dev:USB_C_Receptacle_USB2.0 J1
+L Connector:USB_C_Receptacle_USB2.0 J1
 U 1 1 5F19076D
 P 1100 6250
 F 0 "J1" H 1207 7117 50  0000 C CNN
 F 1 "~" H 1207 7026 50  0001 C CNN
-F 2 "stm32dev:USB_C_Receptacle_HRO_TYPE-C-31-M-12" H 1250 6250 50  0001 C CNN
-F 3 "1811131825_Korean-Hroparts-Elec-TYPE-C-31-M-12_C165948.pdf" H 1250 6250 50  0001 C CNN
-F 4 "C165948" H 1100 6250 50  0001 C CNN "LCSC"
+F 2 "Connector_USB:USB_C_Receptacle_HRO_TYPE-C-31-M-12" H 1250 6250 50  0001 C CNN
+F 3 "https://datasheet.lcsc.com/szlcsc/1811101520_Jing-Extension-of-the-Electronic-Co-C167321_C167321.pdf" H 1250 6250 50  0001 C CNN
+F 4 "C167321" H 1100 6250 50  0001 C CNN "LCSC"
 	1    1100 6250
 	1    0    0    -1
@@
 $EndComp
 $Comp
-L stm32dev:TS-1088R-02526 SW?
+L Switch:SW_Push SW?
 U 1 1 5F1C1C5D
 P 2250 2450
@@
 F 1 "~" H 2450 2550 50  0000 C CNN
 F 2 "stm32dev:TS-1088R-02526" H 2250 2650 50  0001 C CNN
-F 3 "https://datasheet.lcsc.com/szlcsc/1912111437_XUNPU-TS-1088R-02526_C455281.pdf" H 2250 2650 50  0001 C CNN
+F 3 "https://datasheet.lcsc.com/szlcsc/1901111503_XKB-Enterprise-TS-1187A-B-A-B_C318884.pdf" H 2250 2650 50  0001 C CNN
 F 4 "C455281" H 2250 2450 50  0001 C CNN "LCSC"
 	1    2250 2450
@@
 Wire Wire Line
 	6650 4500 6750 4500
+$Comp
+L Device:D_Schottky D?
+U 1 1 60776400
+P 14400 1000
+F 0 "D?" H 14400 875 50  0000 C CNN
+F 1 "~" H 14400 874 50  0000 C CNN
+F 2 "Diode_SMD:D_SOD-123" H 14400 1000 50  0001 C CNN
+F 3 "~" H 14400 1000 50  0001 C CNN
+F 4 "C8598" H 14400 1000 50  0001 C CNN "LCSC"
+	1    14400 1000
+	-1   0    0    1
+$EndComp
+$Comp
+L power:GND #PWR?
+U 1 1 60776406
+P 12900 2700
+F 0 "#PWR?" H 12900 2450 50  0001 C CNN
+F 1 "GND" H 12905 2527 50  0000 C CNN
+F 2 "" H 12900 2700 50  0001 C CNN
+F 3 "" H 12900 2700 50  0001 C CNN
+	1    12900 2700
+	1    0    0    -1
+$EndComp
+Wire Wire Line
+	13500 1500 13600 1500
+Wire Wire Line
+	13500 1600 13600 1600
+Wire Wire Line
+	13600 1600 13600 1500
+Connection ~ 13600 1500
+Wire Wire Line
+	13500 1800 13600 1800
+Wire Wire Line
+	13600 1800 13600 1700
+Connection ~ 13600 1700
+Wire Wire Line
+	13600 1700 13500 1700
+Wire Wire Line
+	13500 1000 13750 1000
+Wire Wire Line
+	14550 1300 13500 1300
+Wire Wire Line
+	13500 1200 14550 1200
+Wire Wire Line
+	12900 2500 12900 2600
+Wire Wire Line
+	12600 2500 12600 2600
+Wire Wire Line
+	12600 2600 12900 2600
+Connection ~ 12900 2600
+Wire Wire Line
+	12900 2600 12900 2700
+$Comp
+L power:VBUS #PWR?
+U 1 1 6077641C
+P 14100 900
+F 0 "#PWR?" H 14100 750 50  0001 C CNN
+F 1 "VBUS" H 14115 1073 50  0000 C CNN
+F 2 "" H 14100 900 50  0001 C CNN
+F 3 "" H 14100 900 50  0001 C CNN
+	1    14100 900
+	1    0    0    -1
+$EndComp
+Wire Wire Line
+	14550 1000 14700 1000
+Wire Wire Line
+	15050 1000 15050 900
+Wire Wire Line
+	14100 900  14100 1000
+Connection ~ 14100 1000
+Wire Wire Line
+	14100 1000 14250 1000
+$Comp
+L power:PWR_FLAG #FLG?
+U 1 1 60776427
+P 13750 900
+F 0 "#FLG?" H 13750 975 50  0001 C CNN
+F 1 "PWR_FLAG" H 13750 1073 50  0001 C CNN
+F 2 "" H 13750 900 50  0001 C CNN
+F 3 "~" H 13750 900 50  0001 C CNN
+	1    13750 900
+	1    0    0    -1
+$EndComp
+Wire Wire Line
+	13750 900  13750 1000
+Connection ~ 13750 1000
+Wire Wire Line
+	13750 1000 14100 1000
+$Comp
+L power:PWR_FLAG #FLG?
+U 1 1 60776430
+P 14700 900
+F 0 "#FLG?" H 14700 975 50  0001 C CNN
+F 1 "PWR_FLAG" H 14700 1073 50  0001 C CNN
+F 2 "" H 14700 900 50  0001 C CNN
+F 3 "~" H 14700 900 50  0001 C CNN
+	1    14700 900
+	1    0    0    -1
+$EndComp
+Wire Wire Line
+	14700 900  14700 1000
+Connection ~ 14700 1000
+Wire Wire Line
+	14700 1000 15050 1000
+$Comp
+L lifeline:USB_C_Receptacle_USB2.0 J?
+U 1 1 6077643B
+P 12900 1600
+F 0 "J?" H 12550 2350 50  0000 C CNN
+F 1 "USB_C_Receptacle_USB2.0" H 13007 2376 50  0001 C CNN
+F 2 "lifeline:USB_C_Receptacle_HRO_TYPE-C-31-M-12" H 13050 1600 50  0001 C CNN
+F 3 "https://datasheet.lcsc.com/szlcsc/1811101520_Jing-Extension-of-the-Electronic-Co-C167321_C167321.pdf" H 13050 1600 50  0001 C CNN
+F 4 "C167321" H 12900 1600 50  0001 C CNN "LCSCAlt"
+F 5 "C165948" H 12900 1600 50  0001 C CNN "LCSC"
+	1    12900 1600
+	1    0    0    -1
+$EndComp
+Text GLabel 14550 1200 2    50   Input ~ 0
+CC1
+Text GLabel 14550 1300 2    50   Input ~ 0
+CC2
+$Comp
+L power:VDC #PWR?
+U 1 1 60776443
+P 15050 900
+F 0 "#PWR?" H 15050 800 50  0001 C CNN
+F 1 "VDC" H 15065 1073 50  0000 C CNN
+F 2 "" H 15050 900 50  0001 C CNN
+F 3 "" H 15050 900 50  0001 C CNN
+	1    15050 900
+	1    0    0    -1
+$EndComp
+$Comp
+L Power_Protection:SP0502BAHT D?
+U 1 1 6077644A
+P 15250 2050
+F 0 "D?" H 15350 2200 50  0000 L CNN
+F 1 "PSM712" H 15300 1900 50  0000 L CNN
+F 2 "Package_TO_SOT_SMD:SOT-23" H 15475 2000 50  0001 L CNN
+F 3 "https://datasheet.lcsc.com/szlcsc/ProTek-Devices-PSM712-LF-T7_C32677.pdf" H 15375 2175 50  0001 C CNN
+F 4 "C32677" H 15250 2050 50  0001 C CNN "LCSC"
+	1    15250 2050
+	1    0    0    -1
+$EndComp
+$Comp
+L power:GND #PWR?
+U 1 1 60776450
+P 15250 2350
+F 0 "#PWR?" H 15250 2100 50  0001 C CNN
+F 1 "GND" H 15255 2177 50  0000 C CNN
+F 2 "" H 15250 2350 50  0001 C CNN
+F 3 "" H 15250 2350 50  0001 C CNN
+	1    15250 2350
+	1    0    0    -1
+$EndComp
+Wire Wire Line
+	15250 2350 15250 2250
+Text GLabel 16200 1500 2    50   Input ~ 0
+HUDM
+Text GLabel 16200 1700 2    50   Input ~ 0
+HUDP
+Wire Wire Line
+	16200 1500 15150 1500
+Wire Wire Line
+	15150 1500 15150 1850
+Wire Wire Line
+	15350 1700 15350 1850
+Wire Wire Line
+	16200 1700 15350 1700
+Wire Wire Line
+	13600 1500 15150 1500
+Connection ~ 15150 1500
+Wire Wire Line
+	13600 1700 15350 1700
+Connection ~ 15350 1700
+$Comp
+L Connector:TestPoint TP?
+U 1 1 60776461
+P 15150 1400
+F 0 "TP?" H 15200 1450 50  0000 L CNN
+F 1 "~" H 15208 1427 50  0000 L CNN
+F 2 "TestPoint:TestPoint_Pad_1.5x1.5mm" H 15350 1400 50  0001 C CNN
+F 3 "~" H 15350 1400 50  0001 C CNN
+	1    15150 1400
+	1    0    0    -1
+$EndComp
+$Comp
+L Connector:TestPoint TP?
+U 1 1 60776467
+P 15350 1400
+F 0 "TP?" H 15400 1450 50  0000 L CNN
+F 1 "~" H 15408 1427 50  0000 L CNN
+F 2 "TestPoint:TestPoint_Pad_1.5x1.5mm" H 15550 1400 50  0001 C CNN
+F 3 "~" H 15550 1400 50  0001 C CNN
+	1    15350 1400
+	1    0    0    -1
+$EndComp
+Wire Wire Line
+	15150 1500 15150 1400
+Wire Wire Line
+	15350 1400 15350 1700
 $EndSCHEMATC

Commit message: Hmmm
Parts:
- removed D?: ~, Diode_SMD:D_SOD-123, symbol Device:D_Schottky
- removed D?: PSM712, Package_TO_SOT_SMD:SOT-23, symbol Power_Protection:SP0502BAHT
- removed J?: USB_C_Receptacle_USB2.0, lifeline:USB_C_Receptacle_HRO_TYPE-C-31-M-12, symbol lifeline:USB_C_Receptacle_USB2.0
- removed TP? (x2): ~, TestPoint:TestPoint_Pad_1.5x1.5mm, symbol Connector:TestPoint
- added H1, H2, H3, H4: ~, MountingHole:MountingHole_2.2mm_M2, symbol Mechanical:MountingHole
- J1: LCSC C167321 -> C165948
Connections:
- net labels removed: CC1, CC2, HUDM, HUDP, VDC
- wire segments 317 -> 287
Changed lines of the file:
@@
 F 2 "Connector_USB:USB_C_Receptacle_HRO_TYPE-C-31-M-12" H 1250 6250 50  0001 C CNN
 F 3 "https://datasheet.lcsc.com/szlcsc/1811101520_Jing-Extension-of-the-Electronic-Co-C167321_C167321.pdf" H 1250 6250 50  0001 C CNN
-F 4 "C167321" H 1100 6250 50  0001 C CNN "LCSC"
+F 4 "C165948" H 1100 6250 50  0001 C CNN "LCSC"
 	1    1100 6250
 	1    0    0    -1
@@
 	6650 4500 6750 4500
 $Comp
-L Device:D_Schottky D?
-U 1 1 60776400
-P 14400 1000
-F 0 "D?" H 14400 875 50  0000 C CNN
-F 1 "~" H 14400 874 50  0000 C CNN
-F 2 "Diode_SMD:D_SOD-123" H 14400 1000 50  0001 C CNN
-F 3 "~" H 14400 1000 50  0001 C CNN
-F 4 "C8598" H 14400 1000 50  0001 C CNN "LCSC"
-	1    14400 1000
-	-1   0    0    1
-$EndComp
-$Comp
-L power:GND #PWR?
-U 1 1 60776406
-P 12900 2700
-F 0 "#PWR?" H 12900 2450 50  0001 C CNN
-F 1 "GND" H 12905 2527 50  0000 C CNN
-F 2 "" H 12900 2700 50  0001 C CNN
-F 3 "" H 12900 2700 50  0001 C CNN
-	1    12900 2700
-	1    0    0    -1
-$EndComp
-Wire Wire Line
-	13500 1500 13600 1500
-Wire Wire Line
-	13500 1600 13600 1600
-Wire Wire Line
-	13600 1600 13600 1500
-Connection ~ 13600 1500
-Wire Wire Line
-	13500 1800 13600 1800
-Wire Wire Line
-	13600 1800 13600 1700
-Connection ~ 13600 1700
-Wire Wire Line
-	13600 1700 13500 1700
-Wire Wire Line
-	13500 1000 13750 1000
-Wire Wire Line
-	14550 1300 13500 1300
-Wire Wire Line
-	13500 1200 14550 1200
-Wire Wire Line
-	12900 2500 12900 2600
-Wire Wire Line
-	12600 2500 12600 2600
-Wire Wire Line
-	12600 2600 12900 2600
-Connection ~ 12900 2600
-Wire Wire Line
-	12900 2600 12900 2700
-$Comp
-L power:VBUS #PWR?
-U 1 1 6077641C
-P 14100 900
-F 0 "#PWR?" H 14100 750 50  0001 C CNN
-F 1 "VBUS" H 14115 1073 50  0000 C CNN
-F 2 "" H 14100 900 50  0001 C CNN
-F 3 "" H 14100 900 50  0001 C CNN
-	1    14100 900
-	1    0    0    -1
-$EndComp
-Wire Wire Line
-	14550 1000 14700 1000
-Wire Wire Line
-	15050 1000 15050 900
-Wire Wire Line
-	14100 900  14100 1000
-Connection ~ 14100 1000
-Wire Wire Line
-	14100 1000 14250 1000
-$Comp
-L power:PWR_FLAG #FLG?
-U 1 1 60776427
-P 13750 900
-F 0 "#FLG?" H 13750 975 50  0001 C CNN
-F 1 "PWR_FLAG" H 13750 1073 50  0001 C CNN
-F 2 "" H 13750 900 50  0001 C CNN
-F 3 "~" H 13750 900 50  0001 C CNN
-	1    13750 900
-	1    0    0    -1
-$EndComp
-Wire Wire Line
-	13750 900  13750 1000
-Connection ~ 13750 1000
-Wire Wire Line
-	13750 1000 14100 1000
-$Comp
-L power:PWR_FLAG #FLG?
-U 1 1 60776430
-P 14700 900
-F 0 "#FLG?" H 14700 975 50  0001 C CNN
-F 1 "PWR_FLAG" H 14700 1073 50  0001 C CNN
-F 2 "" H 14700 900 50  0001 C CNN
-F 3 "~" H 14700 900 50  0001 C CNN
-	1    14700 900
-	1    0    0    -1
-$EndComp
-Wire Wire Line
-	14700 900  14700 1000
-Connection ~ 14700 1000
-Wire Wire Line
-	14700 1000 15050 1000
-$Comp
-L lifeline:USB_C_Receptacle_USB2.0 J?
-U 1 1 6077643B
-P 12900 1600
-F 0 "J?" H 12550 2350 50  0000 C CNN
-F 1 "USB_C_Receptacle_USB2.0" H 13007 2376 50  0001 C CNN
-F 2 "lifeline:USB_C_Receptacle_HRO_TYPE-C-31-M-12" H 13050 1600 50  0001 C CNN
-F 3 "https://datasheet.lcsc.com/szlcsc/1811101520_Jing-Extension-of-the-Electronic-Co-C167321_C167321.pdf" H 13050 1600 50  0001 C CNN
-F 4 "C167321" H 12900 1600 50  0001 C CNN "LCSCAlt"
-F 5 "C165948" H 12900 1600 50  0001 C CNN "LCSC"
-	1    12900 1600
-	1    0    0    -1
-$EndComp
-Text GLabel 14550 1200 2    50   Input ~ 0
-CC1
-Text GLabel 14550 1300 2    50   Input ~ 0
-CC2
-$Comp
-L power:VDC #PWR?
-U 1 1 60776443
-P 15050 900
-F 0 "#PWR?" H 15050 800 50  0001 C CNN
-F 1 "VDC" H 15065 1073 50  0000 C CNN
-F 2 "" H 15050 900 50  0001 C CNN
-F 3 "" H 15050 900 50  0001 C CNN
-	1    15050 900
-	1    0    0    -1
-$EndComp
-$Comp
-L Power_Protection:SP0502BAHT D?
-U 1 1 6077644A
-P 15250 2050
-F 0 "D?" H 15350 2200 50  0000 L CNN
-F 1 "PSM712" H 15300 1900 50  0000 L CNN
-F 2 "Package_TO_SOT_SMD:SOT-23" H 15475 2000 50  0001 L CNN
-F 3 "https://datasheet.lcsc.com/szlcsc/ProTek-Devices-PSM712-LF-T7_C32677.pdf" H 15375 2175 50  0001 C CNN
-F 4 "C32677" H 15250 2050 50  0001 C CNN "LCSC"
-	1    15250 2050
-	1    0    0    -1
-$EndComp
-$Comp
-L power:GND #PWR?
-U 1 1 60776450
-P 15250 2350
-F 0 "#PWR?" H 15250 2100 50  0001 C CNN
-F 1 "GND" H 15255 2177 50  0000 C CNN
-F 2 "" H 15250 2350 50  0001 C CNN
-F 3 "" H 15250 2350 50  0001 C CNN
-	1    15250 2350
-	1    0    0    -1
-$EndComp
-Wire Wire Line
-	15250 2350 15250 2250
-Text GLabel 16200 1500 2    50   Input ~ 0
-HUDM
-Text GLabel 16200 1700 2    50   Input ~ 0
-HUDP
-Wire Wire Line
-	16200 1500 15150 1500
-Wire Wire Line
-	15150 1500 15150 1850
-Wire Wire Line
-	15350 1700 15350 1850
-Wire Wire Line
-	16200 1700 15350 1700
-Wire Wire Line
-	13600 1500 15150 1500
-Connection ~ 15150 1500
-Wire Wire Line
-	13600 1700 15350 1700
-Connection ~ 15350 1700
-$Comp
-L Connector:TestPoint TP?
-U 1 1 60776461
-P 15150 1400
-F 0 "TP?" H 15200 1450 50  0000 L CNN
-F 1 "~" H 15208 1427 50  0000 L CNN
-F 2 "TestPoint:TestPoint_Pad_1.5x1.5mm" H 15350 1400 50  0001 C CNN
-F 3 "~" H 15350 1400 50  0001 C CNN
-	1    15150 1400
-	1    0    0    -1
-$EndComp
-$Comp
-L Connector:TestPoint TP?
-U 1 1 60776467
-P 15350 1400
-F 0 "TP?" H 15400 1450 50  0000 L CNN
-F 1 "~" H 15408 1427 50  0000 L CNN
-F 2 "TestPoint:TestPoint_Pad_1.5x1.5mm" H 15550 1400 50  0001 C CNN
-F 3 "~" H 15550 1400 50  0001 C CNN
-	1    15350 1400
-	1    0    0    -1
-$EndComp
-Wire Wire Line
-	15150 1500 15150 1400
-Wire Wire Line
-	15350 1400 15350 1700
+L Mechanical:MountingHole H1
+U 1 1 607011D3
+P 7250 6400
+F 0 "H1" H 7350 6400 50  0000 L CNN
+F 1 "~" H 7350 6355 50  0000 L CNN
+F 2 "MountingHole:MountingHole_2.2mm_M2" H 7250 6400 50  0001 C CNN
+F 3 "~" H 7250 6400 50  0001 C CNN
+	1    7250 6400
+	1    0    0    -1
+$EndComp
+$Comp
+L Mechanical:MountingHole H2
+U 1 1 6070349D
+P 7550 6400
+F 0 "H2" H 7650 6400 50  0000 L CNN
+F 1 "~" H 7650 6355 50  0000 L CNN
+F 2 "MountingHole:MountingHole_2.2mm_M2" H 7550 6400 50  0001 C CNN
+F 3 "~" H 7550 6400 50  0001 C CNN
+	1    7550 6400
+	1    0    0    -1
+$EndComp
+$Comp
+L Mechanical:MountingHole H3
+U 1 1 60704BB5
+P 7850 6400
+F 0 "H3" H 7950 6400 50  0000 L CNN
+F 1 "~" H 7950 6355 50  0000 L CNN
+F 2 "MountingHole:MountingHole_2.2mm_M2" H 7850 6400 50  0001 C CNN
+F 3 "~" H 7850 6400 50  0001 C CNN
+	1    7850 6400
+	1    0    0    -1
+$EndComp
+$Comp
+L Mechanical:MountingHole H4
+U 1 1 60705173
+P 8150 6400
+F 0 "H4" H 8250 6400 50  0000 L CNN
+F 1 "~" H 8250 6355 50  0000 L CNN
+F 2 "MountingHole:MountingHole_2.2mm_M2" H 8150 6400 50  0001 C CNN
+F 3 "~" H 8150 6400 50  0001 C CNN
+	1    8150 6400
+	1    0    0    -1
+$EndComp
 $EndSCHEMATC

Commit message: Hmmmm
Parts:
- D3: value YEL -> GR; LCSC C72038 -> C72043
Changed lines of the file:
@@
 AR Path="/5F1C1C27" Ref="D3"  Part="1"
 F 0 "D3" V 3300 2650 50  0000 R CNN
-F 1 "YEL" V 3100 2700 50  0000 R CNN
+F 1 "GR" V 3100 2650 50  0000 R CNN
 F 2 "LED_SMD:LED_0603_1608Metric" H 3200 2550 50  0001 C CNN
 F 3 "~" H 3200 2550 50  0001 C CNN
-F 4 "C72038" V 3200 2550 50  0001 C CNN "LCSC"
+F 4 "C72043" V 3200 2550 50  0001 C CNN "LCSC"
 	1    3200 2550
 	0    1    -1   0
@@
 AR Path="/5F1C1C45" Ref="D4"  Part="1"
 F 0 "D4" V 3550 2650 50  0000 R CNN
-F 1 "BLUE" V 3350 2700 50  0000 R CNN
+F 1 "BLUE" V 3350 2750 50  0000 R CNN
 F 2 "LED_SMD:LED_0603_1608Metric" H 3450 2550 50  0001 C CNN
 F 3 "~" H 3450 2550 50  0001 C CNN

Commit message: Hmmm
Parts:
- R1, R5: value NM -> 10k; LCSC (none) -> C25531
Changed lines of the file:
@@
 AR Path="/5F1C1C2E" Ref="R1"  Part="1"
 F 0 "R1" H 1550 2600 50  0000 C CNN
-F 1 "NM" H 1550 2300 50  0000 C CNN
+F 1 "10k" H 1550 2300 50  0000 C CNN
 F 2 "Resistor_SMD:R_0402_1005Metric" V 1380 2450 50  0001 C CNN
 F 3 "~" H 1450 2450 50  0001 C CNN
-F 4 "" V 1450 2450 50  0001 C CNN "LCSC"
+F 4 "C25531" V 1450 2450 50  0001 C CNN "LCSC"
 	1    1450 2450
 	1    0    0    -1
@@
 AR Path="/5F1C1C83" Ref="R5"  Part="1"
 F 0 "R5" H 2350 3100 50  0000 C CNN
-F 1 "NM" H 2350 2800 50  0000 C CNN
+F 1 "10k" H 2350 2800 50  0000 C CNN
 F 2 "Resistor_SMD:R_0402_1005Metric" V 2180 2950 50  0001 C CNN
 F 3 "~" H 2250 2950 50  0001 C CNN
-F 4 "" V 2250 2950 50  0001 C CNN "LCSC"
+F 4 "C25531" V 2250 2950 50  0001 C CNN "LCSC"
 	1    2250 2950
 	1    0    0    -1

Commit message: Hmmmm
Parts:
- removed D1: WS2812B-Mini, stm32dev:LED_WS2812B_MINI_3.5x3.5mm_P1.9mm, symbol stm32dev:WS2812B-Mini
- added D1: WS2812C-2020, stm32dev:LED_WS2812C-2020, symbol stm32dev:WS2812C-2020
- J1: symbol Connector:USB_C_Receptacle_USB2.0 -> stm32dev:USB_C_Receptacle_USB2.0
Changed lines of the file:
@@
 	3600 4350 3500 4350
-$Comp
-L stm32dev:WS2812B-Mini D1
-U 1 1 620C7EB0
-P 1450 4250
-F 0 "D1" H 1794 4296 50  0000 L CNN
-F 1 "WS2812B-Mini" H 1794 4205 50  0000 L CNN
-F 2 "stm32dev:LED_WS2812B_MINI_3.5x3.5mm_P1.9mm" H 1500 3950 50  0001 L TNN
-F 3 "https://cdn-shop.adafruit.com/datasheets/WS2812B.pdf" H 1550 3875 50  0001 L TNN
-F 4 "C114583" H 1450 4250 50  0001 C CNN "LCSC"
-	1    1450 4250
-	1    0    0    -1
-$EndComp
 $Comp
 L power:GND #PWR07
@@
 $EndComp
 $Comp
-L Connector:USB_C_Receptacle_USB2.0 J1
+L stm32dev:USB_C_Receptacle_USB2.0 J1
 U 1 1 5F19076D
 P 1100 6250
@@
 	1    0    0    -1
 $EndComp
+$Comp
+L stm32dev:WS2812C-2020 D1
+U 1 1 60BE2717
+P 1450 4250
+F 0 "D1" H 1794 4296 50  0000 L CNN
+F 1 "WS2812C-2020" H 1794 4205 50  0000 L CNN
+F 2 "stm32dev:LED_WS2812C-2020" H 1500 3950 50  0001 L TNN
+F 3 "https://ipfs-pin.com/ipfs/QmUrWWQTAtUDvCNqULeBaKaw2HwTcne6zNz3L68ZhahRnx/WS2812C-2020_361_V1.0_EN_20031610354448.pdf" H 1550 3875 50  0001 L TNN
+F 4 "C965556" H 1700 3850 50  0001 C CNN "LCSC"
+	1    1450 4250
+	1    0    0    -1
+$EndComp

Commit message: Hmmm
Parts:
- R1, R5: LCSC C25531 -> C25744
Changed lines of the file:
@@
 F 2 "Resistor_SMD:R_0402_1005Metric" V 1380 2450 50  0001 C CNN
 F 3 "~" H 1450 2450 50  0001 C CNN
-F 4 "C25531" V 1450 2450 50  0001 C CNN "LCSC"
+F 4 "C25744" V 1450 2450 50  0001 C CNN "LCSC"
 	1    1450 2450
 	1    0    0    -1
@@
 F 2 "Resistor_SMD:R_0402_1005Metric" V 2180 2950 50  0001 C CNN
 F 3 "~" H 2250 2950 50  0001 C CNN
-F 4 "C25531" V 2250 2950 50  0001 C CNN "LCSC"
+F 4 "C25744" V 2250 2950 50  0001 C CNN "LCSC"
 	1    2250 2950
 	1    0    0    -1

Commit message: Hmmmm
Parts:
- added C14: 100nF, Capacitor_SMD:C_0402_1005Metric, symbol Device:C
- added D5, D6, D7: WS2812C, stm32dev:LED_WS2812C-2020, symbol stm32dev:WS2812C-2020
- added U3: W25Q128JVS, Package_SO:SOIC-8_5.23x5.23mm_P1.27mm, symbol Memory_Flash:W25Q128JVS
- D1: value WS2812C-2020 -> WS2812C
Connections:
- net labels added: PB3
- net labels removed: SWO
- wire segments 287 -> 314
Other:
- note removed: "Internal pull-up"
- moved on the sheet: C10, C11, C12, C13, C9, J3, U2, Y1
