File: pcb/_autosave-stm32dev.sch (KiCad schematic (older format))
At the start: 35 parts, among them J3 Micro_SD_Card_Det, U1 XC6206P332MR, U2 STM32F405RGTx, Y1 16 MHz

Commit message: Hmmmmm
Parts:
- added D?: ~, Diode_SMD:D_SOD-123, symbol Device:D_Schottky
- added D?: PSM712, Package_TO_SOT_SMD:SOT-23, symbol Power_Protection:SP0502BAHT
- added J?: USB_C_Receptacle_USB2.0, lifeline:USB_C_Receptacle_HRO_TYPE-C-31-M-12, symbol lifeline:USB_C_Receptacle_USB2.0
- added TP? (x2): ~, TestPoint:TestPoint_Pad_1.5x1.5mm, symbol Connector:TestPoint
- SW2: footprint Button_Switch_SMD:SW_SPST_TL3342 -> stm32dev:TS-1088R-02526; LCSC C318887 -> C455281
Connections:
- net labels added: CC1, CC2, HUDM, HUDP, VDC
- wire segments 287 -> 317
Changed lines of the file:
@@
 F 0 "SW2" H 2150 2550 50  0000 C CNN
 F 1 "~" H 2450 2550 50  0000 C CNN
-F 2 "Button_Switch_SMD:SW_SPST_TL3342" H 2250 2650 50  0001 C CNN
+F 2 "stm32dev:TS-1088R-02526" H 2250 2650 50  0001 C CNN
 F 3 "https://datasheet.lcsc.com/szlcsc/1901111503_XKB-Enterprise-TS-1187A-B-A-B_C318884.pdf" H 2250 2650 50  0001 C CNN
-F 4 "C318887" H 2250 2450 50  0001 C CNN "LCSC"
+F 4 "C455281" H 2250 2450 50  0001 C CNN "LCSC"
 	1    2250 2450
 	0    -1   -1   0
@@
 Wire Wire Line
 	6650 4500 6750 4500
+$Comp
+L Device:D_Schottky D?
+U 1 1 60776400
+P 14400 1000
+F 0 "D?" H 14400 875 50  0000 C CNN
+F 1 "~" H 14400 874 50  0000 C CNN
+F 2 "Diode_SMD:D_SOD-123" H 14400 1000 50  0001 C CNN
+F 3 "~" H 14400 1000 50  0001 C CNN
+F 4 "C8598" H 14400 1000 50  0001 C CNN "LCSC"
+	1    14400 1000
+	-1   0    0    1
+$EndComp
+$Comp
+L power:GND #PWR?
+U 1 1 60776406
+P 12900 2700
+F 0 "#PWR?" H 12900 2450 50  0001 C CNN
+F 1 "GND" H 12905 2527 50  0000 C CNN
+F 2 "" H 12900 2700 50  0001 C CNN
+F 3 "" H 12900 2700 50  0001 C CNN
+	1    12900 2700
+	1    0    0    -1
+$EndComp
+Wire Wire Line
+	13500 1500 13600 1500
+Wire Wire Line
+	13500 1600 13600 1600
+Wire Wire Line
+	13600 1600 13600 1500
+Connection ~ 13600 1500
+Wire Wire Line
+	13500 1800 13600 1800
+Wire Wire Line
+	13600 1800 13600 1700
+Connection ~ 13600 1700
+Wire Wire Line
+	13600 1700 13500 1700
+Wire Wire Line
+	13500 1000 13750 1000
+Wire Wire Line
+	14550 1300 13500 1300
+Wire Wire Line
+	13500 1200 14550 1200
+Wire Wire Line
+	12900 2500 12900 2600
+Wire Wire Line
+	12600 2500 12600 2600
+Wire Wire Line
+	12600 2600 12900 2600
+Connection ~ 12900 2600
+Wire Wire Line
+	12900 2600 12900 2700
+$Comp
+L power:VBUS #PWR?
+U 1 1 6077641C
+P 14100 900
+F 0 "#PWR?" H 14100 750 50  0001 C CNN
+F 1 "VBUS" H 14115 1073 50  0000 C CNN
+F 2 "" H 14100 900 50  0001 C CNN
+F 3 "" H 14100 900 50  0001 C CNN
+	1    14100 900
+	1    0    0    -1
+$EndComp
+Wire Wire Line
+	14550 1000 14700 1000
+Wire Wire Line
+	15050 1000 15050 900
+Wire Wire Line
+	14100 900  14100 1000
+Connection ~ 14100 1000
+Wire Wire Line
+	14100 1000 14250 1000
+$Comp
+L power:PWR_FLAG #FLG?
+U 1 1 60776427
+P 13750 900
+F 0 "#FLG?" H 13750 975 50  0001 C CNN
+F 1 "PWR_FLAG" H 13750 1073 50  0001 C CNN
+F 2 "" H 13750 900 50  0001 C CNN
+F 3 "~" H 13750 900 50  0001 C CNN
+	1    13750 900
+	1    0    0    -1
+$EndComp
+Wire Wire Line
+	13750 900  13750 1000
+Connection ~ 13750 1000
+Wire Wire Line
+	13750 1000 14100 1000
+$Comp
+L power:PWR_FLAG #FLG?
+U 1 1 60776430
+P 14700 900
+F 0 "#FLG?" H 14700 975 50  0001 C CNN
+F 1 "PWR_FLAG" H 14700 1073 50  0001 C CNN
+F 2 "" H 14700 900 50  0001 C CNN
+F 3 "~" H 14700 900 50  0001 C CNN
+	1    14700 900
+	1    0    0    -1
+$EndComp
+Wire Wire Line
+	14700 900  14700 1000
+Connection ~ 14700 1000
+Wire Wire Line
+	14700 1000 15050 1000
+$Comp
+L lifeline:USB_C_Receptacle_USB2.0 J?
+U 1 1 6077643B
+P 12900 1600
+F 0 "J?" H 12550 2350 50  0000 C CNN
+F 1 "USB_C_Receptacle_USB2.0" H 13007 2376 50  0001 C CNN
+F 2 "lifeline:USB_C_Receptacle_HRO_TYPE-C-31-M-12" H 13050 1600 50  0001 C CNN
+F 3 "https://datasheet.lcsc.com/szlcsc/1811101520_Jing-Extension-of-the-Electronic-Co-C167321_C167321.pdf" H 13050 1600 50  0001 C CNN
+F 4 "C167321" H 12900 1600 50  0001 C CNN "LCSCAlt"
+F 5 "C165948" H 12900 1600 50  0001 C CNN "LCSC"
+	1    12900 1600
+	1    0    0    -1
+$EndComp
+Text GLabel 14550 1200 2    50   Input ~ 0
+CC1
+Text GLabel 14550 1300 2    50   Input ~ 0
+CC2
+$Comp
+L power:VDC #PWR?
+U 1 1 60776443
+P 15050 900
+F 0 "#PWR?" H 15050 800 50  0001 C CNN
+F 1 "VDC" H 15065 1073 50  0000 C CNN
+F 2 "" H 15050 900 50  0001 C CNN
+F 3 "" H 15050 900 50  0001 C CNN
+	1    15050 900
+	1    0    0    -1
+$EndComp
+$Comp
+L Power_Protection:SP0502BAHT D?
+U 1 1 6077644A
+P 15250 2050
+F 0 "D?" H 15350 2200 50  0000 L CNN
+F 1 "PSM712" H 15300 1900 50  0000 L CNN
+F 2 "Package_TO_SOT_SMD:SOT-23" H 15475 2000 50  0001 L CNN
+F 3 "https://datasheet.lcsc.com/szlcsc/ProTek-Devices-PSM712-LF-T7_C32677.pdf" H 15375 2175 50  0001 C CNN
+F 4 "C32677" H 15250 2050 50  0001 C CNN "LCSC"
+	1    15250 2050
+	1    0    0    -1
+$EndComp
+$Comp
+L power:GND #PWR?
+U 1 1 60776450
+P 15250 2350
+F 0 "#PWR?" H 15250 2100 50  0001 C CNN
+F 1 "GND" H 15255 2177 50  0000 C CNN
+F 2 "" H 15250 2350 50  0001 C CNN
+F 3 "" H 15250 2350 50  0001 C CNN
+	1    15250 2350
+	1    0    0    -1
+$EndComp
+Wire Wire Line
+	15250 2350 15250 2250
+Text GLabel 16200 1500 2    50   Input ~ 0
+HUDM
+Text GLabel 16200 1700 2    50   Input ~ 0
+HUDP
+Wire Wire Line
+	16200 1500 15150 1500
+Wire Wire Line
+	15150 1500 15150 1850
+Wire Wire Line
+	15350 1700 15350 1850
+Wire Wire Line
+	16200 1700 15350 1700
+Wire Wire Line
+	13600 1500 15150 1500
+Connection ~ 15150 1500
+Wire Wire Line
+	13600 1700 15350 1700
+Connection ~ 15350 1700
+$Comp
+L Connector:TestPoint TP?
+U 1 1 60776461
+P 15150 1400
+F 0 "TP?" H 15200 1450 50  0000 L CNN
+F 1 "~" H 15208 1427 50  0000 L CNN
+F 2 "TestPoint:TestPoint_Pad_1.5x1.5mm" H 15350 1400 50  0001 C CNN
+F 3 "~" H 15350 1400 50  0001 C CNN
+	1    15150 1400
+	1    0    0    -1
+$EndComp
+$Comp
+L Connector:TestPoint TP?
+U 1 1 60776467
+P 15350 1400
+F 0 "TP?" H 15400 1450 50  0000 L CNN
+F 1 "~" H 15408 1427 50  0000 L CNN
+F 2 "TestPoint:TestPoint_Pad_1.5x1.5mm" H 15550 1400 50  0001 C CNN
+F 3 "~" H 15550 1400 50  0001 C CNN
+	1    15350 1400
+	1    0    0    -1
+$EndComp
+Wire Wire Line
+	15150 1500 15150 1400
+Wire Wire Line
+	15350 1400 15350 1700
 $EndSCHEMATC
